File: RPi_Zero_pHat_Template-master/In_Out.sch (KiCad schematic (older format))
At the start: 18 parts, among them J3 DHT22 Conn, J4 HD38 Conn, J5 120VAC, J6 R_Si, J7 Ventilador, J8 Bomba Agua, J9 Tira LED, Q1 BT136-500, Q2 2N2222A, Q3 2N2222A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

Commit message: Archivos KiCad
Parts:
- added D1, D2: 1N4004, Diode_THT:D_DO-41_SOD81_P10.16mm_Horizontal, symbol Diode:1N4004
- added R7: 1k, Resistor_SMD:R_0805_2012Metric, symbol Device:R
Connections:
- net labels added: 120VAC
- wire segments 28 -> 42
Other:
- moved on the sheet: J7, J8, J9, R5, R6, U8

Commit message: Archivos KiCad
Parts:
- added R10: 1k, Resistor_SMD:R_0805_2012Metric, symbol Device:R
Changed lines of the file:
@@
 Wire Wire Line
 	2150 2850 2500 2850
+$Comp
+L Device:R R10
+U 1 1 60786FB1
+P 4850 2500
+F 0 "R10" V 4643 2500 50  0000 C CNN
+F 1 "1k" V 4734 2500 50  0000 C CNN
+F 2 "Resistor_SMD:R_0805_2012Metric" V 4780 2500 50  0001 C CNN
+F 3 "~" H 4850 2500 50  0001 C CNN
+	1    4850 2500
+	0    1    1    0
+$EndComp
 $EndSCHEMATC

Commit message: Archivos KiCad
Parts:
- removed D1, D2: 1N4004, Diode_THT:D_DO-41_SOD81_P10.16mm_Horizontal, symbol Diode:1N4004
- removed Q2, Q3: 2N2222A, digikey-footprints:TO-18-3, symbol dk_Transistors-Bipolar-BJT-Single:2N2222A
- removed R10: 1k, Resistor_SMD:R_0805_2012Metric, symbol Device:R
- added D1, D2: 1N4148W-TP, digikey-footprints:SOD-123, symbol dk_Diodes-Rectifiers-Single:1N4148W-TP
- added Q2, Q3: FMMT495TA, digikey-footprints:SOT-23-3, symbol dk_Transistors-Bipolar-BJT-Single:FMMT493TA
- C13: value 0.1uF -> 100nF; footprint Capacitor_SMD:C_0805_2012Metric -> Capacitor_SMD:C_0603_1608Metric
- J3, J4: footprint 520249-2:520249-2 -> RJ9-Conn:520249-2
- Q1: footprint Package_TO_SOT_THT:TO-220-3_Vertical -> Package_TO_SOT_SMD:TO-252-2
- U4: footprint digikey-footprints:TO-220-3 -> digikey-footprints:SOIC-8_W3.9mm
- U5: footprint digikey-footprints:DIP-6_W7.62mm -> OPTOCOUPLER_H11F3SR2M:OPTOCOUPLER_H11F3SR2M
- U8: footprint 2:SOP254P700X210-6N -> TLP:SOP254P700X210-6N

Commit message: Archivos KiCad
Parts:
- added D10, D7, D8, D9: LED, LED_SMD:LED_0805_2012Metric, symbol Device:LED
- added R12, R13, R18: 10k, Resistor_SMD:R_0805_2012Metric, symbol Device:R
- added R14, R15, R16, R17: 1k, Resistor_SMD:R_0805_2012Metric, symbol Device:R
- J7, J8: footprint MOLEX_2:MOLEX_22-29-2021 -> TerminalBlock_Phoenix:TerminalBlock_Phoenix_MKDS-1,5-2-5.08_1x02_P5.08mm_Horizontal
- R4, R7: value 1k -> 220
- R5, R6: value 1k -> 10k
Connections:
- net +5V: now also R18.1
- net GND: now also D10.1 (K), D7.1 (K), D8.1 (K), D9.1 (K), R12.1, R13.1
- net In_Bomba_Agua: now also R16.1
- net In_LEDs: now also R17.1
- net In_Resistencia_Si: now also R14.1
- net In_Ventilador: now also R15.1
- net Out_DHT22: now also R18.2
- net at Q2.1 (B), R5.1: now also R12.2
- net at Q3.1 (B), R6.1: now also R13.2
- new net: D7.2 (A), R14.2
- new net: D8.2 (A), R15.2
- new net: D9.2 (A), R16.2
- new net: D10.2 (A), R17.2
Other:
- moved on the sheet: D1, D2, J5, J6, J7, J8, J9, Q1, Q2, Q3, R3, R4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

Commit message: Archivos KiCad
Parts:
- removed D1, D2: 1N4148W-TP, digikey-footprints:SOD-123, symbol dk_Diodes-Rectifiers-Single:1N4148W-TP
- removed Q2, Q3: FMMT495TA, digikey-footprints:SOT-23-3, symbol dk_Transistors-Bipolar-BJT-Single:FMMT493TA
- added D1, D2: 1N4148WS, Diode_SMD:D_SOD-323, symbol Diode:1N4148WS
- added Q2, Q3: MMBT2222A, digikey-footprints:SOT-23-3, symbol dk_Transistors-Bipolar-BJT-Single:MMBT2222A_Obsolete
- C13: footprint Capacitor_SMD:C_0603_1608Metric -> Capacitor_SMD:C_0201_0603Metric
- R3: footprint Resistor_SMD:R_0805_2012Metric -> Resistor_SMD:R_1206_3216Metric
Connections:
- net +12V: now also D1.1 (K), D2.1 (K)
- net GND: now also Q2.2 (E), Q3.2 (E)
- net at J7.1 (Pin_1): now also D1.2 (A), Q2.3 (C)
- net at J8.1 (Pin_1): now also D2.2 (A), Q3.3 (C)
- net at R12.2, R5.1: now also Q2.1 (B)
- net at R13.2, R6.1: now also Q3.1 (B)
Changed lines of the file:
@@
 F 0 "C13" H 1200 1600 50  0000 L CNN
 F 1 "100nF" H 1200 1500 50  0000 L CNN
-F 2 "Capacitor_SMD:C_0603_1608Metric" H 1488 1350 50  0001 C CNN
+F 2 "Capacitor_SMD:C_0201_0603Metric" H 1488 1350 50  0001 C CNN
 F 3 "~" H 1450 1500 50  0001 C CNN
 	1    1450 1500
@@
 F 0 "R3" V 5343 1200 50  0000 C CNN
 F 1 "180" V 5434 1200 50  0000 C CNN
-F 2 "Resistor_SMD:R_0805_2012Metric" V 5480 1200 50  0001 C CNN
+F 2 "Resistor_SMD:R_1206_3216Metric" V 5480 1200 50  0001 C CNN
 F 3 "~" H 5550 1200 50  0001 C CNN
 	1    5550 1200
@@
 Wire Wire Line
 	9350 3600 9150 3600
-$Comp
-L dk_Diodes-Rectifiers-Single:1N4148W-TP D1
-U 1 1 607C3C93
-P 5750 3100
-F 0 "D1" H 5750 3337 60  0000 C CNN
-F 1 "1N4148W-TP" H 5750 3231 60  0000 C CNN
-F 2 "digikey-footprints:SOD-123" H 5950 3300 60  0001 L CNN
-F 3 "https://www.mccsemi.com/pdf/Products/1N4148W(SOD123).pdf" H 5950 3400 60  0001 L CNN
-F 4 "1N4148WTPMSCT-ND" H 5950 3500 60  0001 L CNN "Digi-Key_PN"
-F 5 "1N4148W-TP" H 5950 3600 60  0001 L CNN "MPN"
-F 6 "Discrete Semiconductor Products" H 5950 3700 60  0001 L CNN "Category"
-F 7 "Diodes - Rectifiers - Single" H 5950 3800 60  0001 L CNN "Family"
-F 8 "https://www.mccsemi.com/pdf/Products/1N4148W(SOD123).pdf" H 5950 3900 60  0001 L CNN "DK_Datasheet_Link"
-F 9 "/product-detail/en/micro-commercial-co/1N4148W-TP/1N4148WTPMSCT-ND/717311" H 5950 4000 60  0001 L CNN "DK_Detail_Page"
-F 10 "DIODE GEN PURP 100V 150MA SOD123" H 5950 4100 60  0001 L CNN "Description"
-F 11 "Micro Commercial Co" H 5950 4200 60  0001 L CNN "Manufacturer"
-F 12 "Active" H 5950 4300 60  0001 L CNN "Status"
-	1    5750 3100
-	1    0    0    -1
-$EndComp
 Wire Wire Line
 	5550 3100 5450 3100
 Wire Wire Line
-	5950 3100 6000 3100
-Wire Wire Line
 	6000 3100 6000 3600
 Wire Wire Line
 	5450 3100 5450 3600
-$Comp
-L dk_Diodes-Rectifiers-Single:1N4148W-TP D2
-U 1 1 607CD147
-P 9100 3150
-F 0 "D2" H 9100 3387 60  0000 C CNN
-F 1 "1N4148W-TP" H 9100 3281 60  0000 C CNN
-F 2 "digikey-footprints:SOD-123" H 9300 3350 60  0001 L CNN
-F 3 "https://www.mccsemi.com/pdf/Products/1N4148W(SOD123).pdf" H 9300 3450 60  0001 L CNN
-F 4 "1N4148WTPMSCT-ND" H 9300 3550 60  0001 L CNN "Digi-Key_PN"
-F 5 "1N4148W-TP" H 9300 3650 60  0001 L CNN "MPN"
-F 6 "Discrete Semiconductor Products" H 9300 3750 60  0001 L CNN "Category"
-F 7 "Diodes - Rectifiers - Single" H 9300 3850 60  0001 L CNN "Family"
-F 8 "https://www.mccsemi.com/pdf/Products/1N4148W(SOD123).pdf" H 9300 3950 60  0001 L CNN "DK_Datasheet_Link"
-F 9 "/product-detail/en/micro-commercial-co/1N4148W-TP/1N4148WTPMSCT-ND/717311" H 9300 4050 60  0001 L CNN "DK_Detail_Page"
-F 10 "DIODE GEN PURP 100V 150MA SOD123" H 9300 4150 60  0001 L CNN "Description"
-F 11 "Micro Commercial Co" H 9300 4250 60  0001 L CNN "Manufacturer"
-F 12 "Active" H 9300 4350 60  0001 L CNN "Status"
-	1    9100 3150
-	1    0    0    -1
-$EndComp
 Wire Wire Line
 	8900 3150 8800 3150
-Wire Wire Line
-	9300 3150 9350 3150
-$Comp
-L dk_Transistors-Bipolar-BJT-Single:FMMT493TA Q2
-U 1 1 607E68CB
-P 5200 3850
-F 0 "Q2" H 5388 3903 60  0000 L CNN
-F 1 "FMMT495TA" H 5388 3797 60  0000 L CNN
-F 2 "digikey-footprints:SOT-23-3" H 5400 4050 60  0001 L CNN
-F 3 "https://www.diodes.com/assets/Datasheets/FMMT493.pdf" H 5400 4150 60  0001 L CNN
-F 4 "FMMT493CT-ND" H 5400 4250 60  0001 L CNN "Digi-Key_PN"
-F 5 "FMMT493TA" H 5400 4350 60  0001 L CNN "MPN"
-F 6 "Discrete Semiconductor Products" H 5400 4450 60  0001 L CNN "Category"
-F 7 "Transistors - Bipolar (BJT) - Single" H 5400 4550 60  0001 L CNN "Family"
-F 8 "https://www.diodes.com/assets/Datasheets/FMMT493.pdf" H 5400 4650 60  0001 L CNN "DK_Datasheet_Link"
-F 9 "/product-detail/en/diodes-incorporated/FMMT493TA/FMMT493CT-ND/92663" H 5400 4750 60  0001 L CNN "DK_Detail_Page"
-F 10 "TRANS NPN 100V 1A SOT23-3" H 5400 4850 60  0001 L CNN "Description"
-F 11 "Diodes Incorporated" H 5400 4950 60  0001 L CNN "Manufacturer"
-F 12 "Active" H 5400 5050 60  0001 L CNN "Status"
-	1    5200 3850
-	1    0    0    -1
-$EndComp
-$Comp
-L dk_Transistors-Bipolar-BJT-Single:FMMT493TA Q3
-U 1 1 607EA985
-P 8600 3850
-F 0 "Q3" H 8788 3903 60  0000 L CNN
-F 1 "FMMT495TA" H 8788 3797 60  0000 L CNN
-F 2 "digikey-footprints:SOT-23-3" H 8800 4050 60  0001 L CNN
-F 3 "https://www.diodes.com/assets/Datasheets/FMMT493.pdf" H 8800 4150 60  0001 L CNN
-F 4 "FMMT493CT-ND" H 8800 4250 60  0001 L CNN "Digi-Key_PN"
-F 5 "FMMT493TA" H 8800 4350 60  0001 L CNN "MPN"
-F 6 "Discrete Semiconductor Products" H 8800 4450 60  0001 L CNN "Category"
-F 7 "Transistors - Bipolar (BJT) - Single" H 8800 4550 60  0001 L CNN "Family"
-F 8 "https://www.diodes.com/assets/Datasheets/FMMT493.pdf" H 8800 4650 60  0001 L CNN "DK_Datasheet_Link"
-F 9 "/product-detail/en/diodes-incorporated/FMMT493TA/FMMT493CT-ND/92663" H 8800 4750 60  0001 L CNN "DK_Detail_Page"
-F 10 "TRANS NPN 100V 1A SOT23-3" H 8800 4850 60  0001 L CNN "Description"
-F 11 "Diodes Incorporated" H 8800 4950 60  0001 L CNN "Manufacturer"
-F 12 "Active" H 8800 5050 60  0001 L CNN "Status"
-	1    8600 3850
-	1    0    0    -1
-$EndComp
 $Comp
 L Device:R R12
@@
 	2850 2850 2700 2850
 Connection ~ 2700 2850
+$Comp
+L Diode:1N4148WS D1
+U 1 1 607FB5A3
+P 5700 3100
+F 0 "D1" H 5700 2883 50  0000 C CNN
+F 1 "1N4148WS" H 5700 2974 50  0000 C CNN
+F 2 "Diode_SMD:D_SOD-323" H 5700 2925 50  0001 C CNN
+F 3 "https://www.vishay.com/docs/85751/1n4148ws.pdf" H 5700 3100 50  0001 C CNN
+	1    5700 3100
+	-1   0    0    1
+$EndComp
+Wire Wire Line
+	5850 3100 6000 3100
+$Comp
+L Diode:1N4148WS D2
+U 1 1 60803048
+P 9050 3150
+F 0 "D2" H 9050 2933 50  0000 C CNN
+F 1 "1N4148WS" H 9050 3024 50  0000 C CNN
+F 2 "Diode_SMD:D_SOD-323" H 9050 2975 50  0001 C CNN
+F 3 "https://www.vishay.com/docs/85751/1n4148ws.pdf" H 9050 3150 50  0001 C CNN
+	1    9050 3150
+	-1   0    0    1
+$EndComp
+Wire Wire Line
+	9200 3150 9350 3150
+$Comp
+L dk_Transistors-Bipolar-BJT-Single:MMBT2222A_Obsolete Q2
+U 1 1 608085CC
+P 5200 3850
+F 0 "Q2" H 5388 3903 60  0000 L CNN
+F 1 "MMBT2222A" H 5388 3797 60  0000 L CNN
+F 2 "digikey-footprints:SOT-23-3" H 5400 4050 60  0001 L CNN
+F 3 "https://media.digikey.com/pdf/Data%20Sheets/Fairchild%20PDFs/MMBT2222A.pdf" H 5400 4150 60  0001 L CNN
+F 4 "MMBT2222AFSCT-ND" H 5400 4250 60  0001 L CNN "Digi-Key_PN"
+F 5 "MMBT2222A" H 5400 4350 60  0001 L CNN "MPN"
+F 6 "Discrete Semiconductor Products" H 5400 4450 60  0001 L CNN "Category"
+F 7 "Transistors - Bipolar (BJT) - Single" H 5400 4550 60  0001 L CNN "Family"
+F 8 "https://media.digikey.com/pdf/Data%20Sheets/Fairchild%20PDFs/MMBT2222A.pdf" H 5400 4650 60  0001 L CNN "DK_Datasheet_Link"
+F 9 "/product-detail/en/on-semiconductor/MMBT2222A/MMBT2222AFSCT-ND/458969" H 5400 4750 60  0001 L CNN "DK_Detail_Page"
+F 10 "TRANS NPN 40V 1A SOT-23" H 5400 4850 60  0001 L CNN "Description"
+F 11 "ON Semiconductor" H 5400 4950 60  0001 L CNN "Manufacturer"
+F 12 "Obsolete NonStock" H 5400 5050 60  0001 L CNN "Status"
+	1    5200 3850
+	1    0    0    -1
+$EndComp
+$Comp
+L dk_Transistors-Bipolar-BJT-Single:MMBT2222A_Obsolete Q3
+U 1 1 6080CE83
+P 8600 3850
+F 0 "Q3" H 8788 3903 60  0000 L CNN
+F 1 "MMBT2222A" H 8788 3797 60  0000 L CNN
+F 2 "digikey-footprints:SOT-23-3" H 8800 4050 60  0001 L CNN
+F 3 "https://media.digikey.com/pdf/Data%20Sheets/Fairchild%20PDFs/MMBT2222A.pdf" H 8800 4150 60  0001 L CNN
+F 4 "MMBT2222AFSCT-ND" H 8800 4250 60  0001 L CNN "Digi-Key_PN"
+F 5 "MMBT2222A" H 8800 4350 60  0001 L CNN "MPN"
+F 6 "Discrete Semiconductor Products" H 8800 4450 60  0001 L CNN "Category"
+F 7 "Transistors - Bipolar (BJT) - Single" H 8800 4550 60  0001 L CNN "Family"
+F 8 "https://media.digikey.com/pdf/Data%20Sheets/Fairchild%20PDFs/MMBT2222A.pdf" H 8800 4650 60  0001 L CNN "DK_Datasheet_Link"
+F 9 "/product-detail/en/on-semiconductor/MMBT2222A/MMBT2222AFSCT-ND/458969" H 8800 4750 60  0001 L CNN "DK_Detail_Page"
+F 10 "TRANS NPN 40V 1A SOT-23" H 8800 4850 60  0001 L CNN "Description"
+F 11 "ON Semiconductor" H 8800 4950 60  0001 L CNN "Manufacturer"
+F 12 "Obsolete NonStock" H 8800 5050 60  0001 L CNN "Status"
+	1    8600 3850
+	1    0    0    -1
+$EndComp
 $EndSCHEMATC

Commit message: Archivos KiCad
Parts:
- C13: footprint Capacitor_SMD:C_0201_0603Metric -> Capacitor_SMD:C_0805_2012Metric
Changed lines of the file:
@@
 F 0 "C13" H 1200 1600 50  0000 L CNN
 F 1 "100nF" H 1200 1500 50  0000 L CNN
-F 2 "Capacitor_SMD:C_0201_0603Metric" H 1488 1350 50  0001 C CNN
+F 2 "Capacitor_SMD:C_0805_2012Metric" H 1488 1350 50  0001 C CNN
 F 3 "~" H 1450 1500 50  0001 C CNN
 	1    1450 1500

Commit message: Archivos KiCad
Parts:
- added H2, H3: MountingHole, MountingHole:MountingHole_3.5mm, symbol Mechanical:MountingHole
- D10: value LED -> LEDs
- D7: value LED -> LED_RSi
- D8: value LED -> LED_Vent
- D9: value LED -> LED_H2O
Connections:
- net 120VAC: now also J5.2 (Pin_2), J6.1 (Pin_1); no longer J5.1 (Pin_1), J6.2 (Pin_2)
- net GNDREF: now also J5.1 (Pin_1); no longer J5.2 (Pin_2)
- net at Q1.2 (A2), R3.1: now also J6.2 (Pin_2); no longer J6.1 (Pin_1)
Other:
- moved on the sheet: J5, J6
Changed lines of the file:
@@
 L Connector:Screw_Terminal_01x02 J6
 U 1 1 6074CBC0
-P 6050 1000
-F 0 "J6" V 6014 812 50  0000 R CNN
-F 1 "R_Si" V 5923 812 50  0000 R CNN
-F 2 "TerminalBlock_Phoenix:TerminalBlock_Phoenix_MKDS-1,5-2-5.08_1x02_P5.08mm_Horizontal" H 6050 1000 50  0001 C CNN
-F 3 "~" H 6050 1000 50  0001 C CNN
-	1    6050 1000
-	0    -1   -1   0
+P 6100 1000
+F 0 "J6" V 6150 1200 50  0000 R CNN
+F 1 "R_Si" V 6050 1250 50  0000 R CNN
+F 2 "TerminalBlock_Phoenix:TerminalBlock_Phoenix_MKDS-1,5-2-5.08_1x02_P5.08mm_Horizontal" H 6100 1000 50  0001 C CNN
+F 3 "~" H 6100 1000 50  0001 C CNN
+	1    6100 1000
+	0    1    -1   0
 $EndComp
 $Comp
 L power:GNDREF #PWR0138
 U 1 1 6073AE44
-P 6850 1200
-F 0 "#PWR0138" H 6850 950 50  0001 C CNN
-F 1 "GNDREF" H 6855 1027 50  0000 C CNN
-F 2 "" H 6850 1200 50  0001 C CNN
-F 3 "" H 6850 1200 50  0001 C CNN
-	1    6850 1200
-	1    0    0    -1
-$EndComp
-$Comp
-L Connector:Screw_Terminal_01x02 J5
-U 1 1 60750E09
-P 6750 1000
-F 0 "J5" V 6714 812 50  0000 R CNN
-F 1 "120VAC" V 6623 812 50  0000 R CNN
-F 2 "TerminalBlock_Phoenix:TerminalBlock_Phoenix_MKDS-1,5-2-5.08_1x02_P5.08mm_Horizontal" H 6750 1000 50  0001 C CNN
-F 3 "~" H 6750 1000 50  0001 C CNN
-	1    6750 1000
-	0    -1   -1   0
-$EndComp
-Wire Wire Line
-	6750 1200 6150 1200
-Wire Wire Line
-	6050 1200 5800 1200
+P 6750 1200
+F 0 "#PWR0138" H 6750 950 50  0001 C CNN
+F 1 "GNDREF" H 6755 1027 50  0000 C CNN
+F 2 "" H 6750 1200 50  0001 C CNN
+F 3 "" H 6750 1200 50  0001 C CNN
+	1    6750 1200
+	1    0    0    -1
+$EndComp
 Wire Wire Line
 	5400 1200 5250 1200
 Wire Wire Line
 	5700 1200 5800 1200
-Connection ~ 5800 1200
 Wire Wire Line
 	5150 1550 5650 1550
@@
 	1    0    0    -1
 $EndComp
-Text Label 6400 1200 0    50   ~ 0
+Text Label 6250 1200 0    50   ~ 0
 120VAC
 $Comp
@@
 AR Path="/6081C49D/608150DB" Ref="D7"  Part="1"
 F 0 "D7" H 4100 2250 50  0000 C CNN
-F 1 "LED" H 4100 2150 50  0000 C CNN
+F 1 "LED_RSi" H 4100 2150 50  0000 C CNN
 F 2 "LED_SMD:LED_0805_2012Metric" H 4100 2000 50  0001 C CNN
 F 3 "~" H 4100 2000 50  0001 C CNN
@@
 AR Path="/6081C49D/6081979C" Ref="D8"  Part="1"
 F 0 "D8" H 4450 4750 50  0000 C CNN
-F 1 "LED" H 4450 4650 50  0000 C CNN
+F 1 "LED_Vent" H 4450 4650 50  0000 C CNN
 F 2 "LED_SMD:LED_0805_2012Metric" H 4450 4500 50  0001 C CNN
 F 3 "~" H 4450 4500 50  0001 C CNN
@@
 AR Path="/6081C49D/6081EC29" Ref="D9"  Part="1"
 F 0 "D9" H 7850 4750 50  0000 C CNN
-F 1 "LED" H 7850 4650 50  0000 C CNN
+F 1 "LED_H2O" H 7850 4650 50  0000 C CNN
 F 2 "LED_SMD:LED_0805_2012Metric" H 7850 4500 50  0001 C CNN
 F 3 "~" H 7850 4500 50  0001 C CNN
@@
 AR Path="/6081C49D/60824789" Ref="D10"  Part="1"
 F 0 "D10" H 8600 2100 50  0000 C CNN
-F 1 "LED" H 8600 2000 50  0000 C CNN
+F 1 "LEDs" H 8600 2000 50  0000 C CNN
 F 2 "LED_SMD:LED_0805_2012Metric" H 8600 1850 50  0001 C CNN
 F 3 "~" H 8600 1850 50  0001 C CNN
@@
 	1    0    0    -1
 $EndComp
+$Comp
+L Mechanical:MountingHole H2
+U 1 1 608467C0
+P 9850 5600
+F 0 "H2" H 9950 5646 50  0000 L CNN
+F 1 "MountingHole" H 9950 5555 50  0000 L CNN
+F 2 "MountingHole:MountingHole_3.5mm" H 9850 5600 50  0001 C CNN
+F 3 "~" H 9850 5600 50  0001 C CNN
+	1    9850 5600
+	1    0    0    -1
+$EndComp
+$Comp
+L Mechanical:MountingHole H3
+U 1 1 60846A18
+P 9850 6000
+F 0 "H3" H 9950 6046 50  0000 L CNN
+F 1 "MountingHole" H 9950 5955 50  0000 L CNN
+F 2 "MountingHole:MountingHole_3.5mm" H 9850 6000 50  0001 C CNN
+F 3 "~" H 9850 6000 50  0001 C CNN
+	1    9850 6000
+	1    0    0    -1
+$EndComp
+$Comp
+L Connector:Screw_Terminal_01x02 J5
+U 1 1 60750E09
+P 6750 1000
+F 0 "J5" V 6750 1200 50  0000 R CNN
+F 1 "120VAC" V 6650 1350 50  0000 R CNN
+F 2 "TerminalBlock_Phoenix:TerminalBlock_Phoenix_MKDS-1,5-2-5.08_1x02_P5.08mm_Horizontal" H 6750 1000 50  0001 C CNN
+F 3 "~" H 6750 1000 50  0001 C CNN
+	1    6750 1000
+	0    1    -1   0
+$EndComp
+Wire Wire Line
+	6100 1200 6650 1200
+Wire Wire Line
+	6000 1200 5800 1200
+Connection ~ 5800 1200
 $EndSCHEMATC

Commit message: Archivos KiCad
Parts:
- removed D1, D2: 1N4148WS, Diode_SMD:D_SOD-323, symbol Diode:1N4148WS
- added D1, D2: MRA4004T3G, Diode_SMD:D_SMA, symbol Diode:MRA4004T3G
Connections:
- net +12V: now also D1.1 (K), D2.1 (K)
- net at J7.1 (Pin_1), Q2.3 (C): now also D1.2 (A)
- net at J8.1 (Pin_1), Q3.3 (C): now also D2.2 (A)
Changed lines of the file:
@@
 	2850 2850 2700 2850
 Connection ~ 2700 2850
-$Comp
-L Diode:1N4148WS D1
-U 1 1 607FB5A3
-P 5700 3100
-F 0 "D1" H 5700 2883 50  0000 C CNN
-F 1 "1N4148WS" H 5700 2974 50  0000 C CNN
-F 2 "Diode_SMD:D_SOD-323" H 5700 2925 50  0001 C CNN
-F 3 "https://www.vishay.com/docs/85751/1n4148ws.pdf" H 5700 3100 50  0001 C CNN
-	1    5700 3100
-	-1   0    0    1
-$EndComp
 Wire Wire Line
 	5850 3100 6000 3100
-$Comp
-L Diode:1N4148WS D2
-U 1 1 60803048
-P 9050 3150
-F 0 "D2" H 9050 2933 50  0000 C CNN
-F 1 "1N4148WS" H 9050 3024 50  0000 C CNN
-F 2 "Diode_SMD:D_SOD-323" H 9050 2975 50  0001 C CNN
-F 3 "https://www.vishay.com/docs/85751/1n4148ws.pdf" H 9050 3150 50  0001 C CNN
-	1    9050 3150
-	-1   0    0    1
-$EndComp
 Wire Wire Line
 	9200 3150 9350 3150
@@
 	6000 1200 5800 1200
 Connection ~ 5800 1200
+$Comp
+L Diode:MRA4004T3G D2
+U 1 1 608B4401
+P 9050 3150
+F 0 "D2" H 9050 2933 50  0000 C CNN
+F 1 "MRA4004T3G" H 9050 3024 50  0000 C CNN
+F 2 "Diode_SMD:D_SMA" H 9050 2975 50  0001 C CNN
+F 3 "http://www.onsemi.com/pub_link/Collateral/MRA4003T3-D.PDF" H 9050 3150 50  0001 C CNN
+	1    9050 3150
+	-1   0    0    1
+$EndComp
+$Comp
+L Diode:MRA4004T3G D1
+U 1 1 608BA0DD
+P 5700 3100
+F 0 "D1" H 5700 2883 50  0000 C CNN
+F 1 "MRA4004T3G" H 5700 2974 50  0000 C CNN
+F 2 "Diode_SMD:D_SMA" H 5700 2925 50  0001 C CNN
+F 3 "http://www.onsemi.com/pub_link/Collateral/MRA4003T3-D.PDF" H 5700 3100 50  0001 C CNN
+	1    5700 3100
+	-1   0    0    1
+$EndComp
 $EndSCHEMATC
