File: RPi_Zero_pHat_Template-master/RPi_Zero_pHat_Template.kicad_pcb (KiCad board)
At the start: 2 copper layers, 105.4 x 72.4 mm, 43 parts, among them J1 POWER_JACK, J2 RPi_GPIO, J3 DHT22 Conn, J4 HD38 Conn, J5 120VAC, J6 R_Si, J7 Ventilador, J8 Bomba Agua, J9 Tira LED, Q1 BT136-500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

Commit message: Archivos KiCad
Parts:
- added D1: 1N4004, Diode_THT:D_DO-41_SOD81_P10.16mm_Horizontal, F.Cu at (143.5, 66.0)
- added D2: 1N4004, Diode_THT:D_DO-41_SOD81_P10.16mm_Horizontal, F.Cu at (143.5, 70.3)
- added R7: 1k, Resistor_SMD:R_0805_2012Metric, F.Cu at (143.5, 45.1)
- C5: value 10nF -> 100nF
- C6: value 1uF -> 10nF
- C8: value 100nF -> 1uF
- moved L1 59.1 mm to (88.2, 64.6)
- moved C4 47.6 mm to (88.2, 70.3)
- moved C8 45.7 mm to (92.6, 70.8)
- moved C5 45.6 mm to (92.7, 67.8)
- moved C7 45.3 mm to (88.2, 73.3)
- moved C12 43.4 mm to (92.6, 73.8)
- moved C1 43.0 mm to (92.7, 64.8)
- moved C6 35.5 mm to (97.2, 64.8)
- moved C11 30.7 mm to (97.2, 67.8)
- moved L2 21.4 mm to (88.2, 67.4)
- moved R2 11.4 mm to (97.0, 73.7)
- moved U1 10.9 mm to (80.3, 68.9)
- moved R1 7.30 mm to (97.0, 70.8)
Connections:
- net /RX renamed /USART1
- net /Sheet6081C49C/Out_DHT22 renamed Net-(J3-Pad2)
- net /TX renamed /USART2
- net Net-(J5-Pad1) renamed /In_Out/120VAC
- C5 pad 1: /Alimentacion/VDDA -> +3V3
- C6 pad 1: /Alimentacion/VDDA -> /STM32/VDDA
- C8 pad 1: +3V3 -> /STM32/VDDA
- J2 pad 32: Net-(J2-Pad32) -> /BOOT
- J2 pad 33: Net-(J2-Pad33) -> /NRST
- J3 pad 1: +5V -> /DHT22
- J3 pad 3: Net-(J3-Pad3) -> GND
- J3 pad 4: GND -> +5V
- J4 pad 1: /Sheet6081C49C/Out_HD38 -> /HD38
- L2 pad 2: /Alimentacion/VDDA -> /STM32/VDDA
- R4 pad 2: /Sheet6081C49C/In_Resistencia_Si -> /Resistencia_Si
- R5 pad 2: /Sheet6081C49C/In_Ventilador -> /Ventilador
- R6 pad 2: /Sheet6081C49C/In_Bomba_Agua -> /Bomba_Agua
- U1 pad 11: Net-(U1-Pad11) -> /Resistencia_Si
- U1 pad 12: Net-(U1-Pad12) -> /Ventilador
- U1 pad 13: Net-(U1-Pad13) -> /Bomba_Agua
- U1 pad 14: Net-(U1-Pad14) -> /LEDs
- U1 pad 15: Net-(U1-Pad15) -> /LM35
- U1 pad 16: Net-(U1-Pad16) -> /HD38
- U1 pad 17: Net-(U1-Pad17) -> /DHT22
- U1 pad 44: Net-(U1-Pad44) -> /BOOT
- U1 pad 7: Net-(U1-Pad7) -> /NRST
- U1 pad 9: /Alimentacion/VDDA -> /STM32/VDDA
- U4 pad 3: /Sheet6081C49C/Out_LM35 -> /LM35
- U8 pad 1: /Sheet6081C49C/In_LEDs -> Net-(R7-Pad1)
- U8 pad 2: Net-(U8-Pad2) -> GND

Commit message: Archivos KiCad
Parts:
- added D3: LED, LED_SMD:LED_0805_2012Metric, F.Cu at (260.4, 143.5)
- added D4: LED, LED_SMD:LED_0805_2012Metric, F.Cu at (261.0, 162.6)
- added D5: LED, LED_SMD:LED_0805_2012Metric, F.Cu at (217.8, 74.3)
- added D6: LED, LED_SMD:LED_0805_2012Metric, F.Cu at (179.1, 97.2)
- added R10: 1k, Resistor_SMD:R_0805_2012Metric, F.Cu at (183.5, 97.1)
- added R11: 1k, Resistor_SMD:R_0805_2012Metric, F.Cu at (217.8, 68.6)
- added R8: 1k, Resistor_SMD:R_0805_2012Metric, F.Cu at (259.7, 139.1)
- added R9: 1k, Resistor_SMD:R_0805_2012Metric, F.Cu at (260.4, 156.2)
- C1, C11, C4, C5, C6, C7: footprint Capacitor_SMD:C_0805_2012Metric -> Capacitor_SMD:C_0603_1608Metric
- C13: value 0.1uF -> 100nF; footprint Capacitor_SMD:C_0805_2012Metric -> Capacitor_SMD:C_0603_1608Metric
- C8: footprint Capacitor_SMD:C_0805_2012Metric -> Capacitor_SMD:C_0402_1005Metric
- D1, D2: value 1N4004 -> 1N4148W-TP; footprint Diode_THT:D_DO-41_SOD81_P10.16mm_Horizontal -> digikey-footprints:SOD-123
- J3, J4: footprint 520249-2:520249-2 -> RJ9-Conn:520249-2
- L1, L2: value L -> 33nH; footprint Inductor_SMD:L_0805_2012Metric -> Inductor_SMD:L_0402_1005Metric
- Q1: footprint Package_TO_SOT_THT:TO-220-3_Vertical -> Package_TO_SOT_SMD:TO-252-2
- Q2, Q3: value 2N2222A -> FMMT495TA; footprint digikey-footprints:TO-18-3 -> digikey-footprints:SOT-23-3
- U4: footprint digikey-footprints:TO-220-3 -> digikey-footprints:SOIC-8_W3.9mm
- U5: footprint digikey-footprints:DIP-6_W7.62mm -> OPTOCOUPLER_H11F3SR2M:OPTOCOUPLER_H11F3SR2M
- U8: footprint 2:SOP254P700X210-6N -> TLP:SOP254P700X210-6N
- moved C2 183.6 mm to (254.0, 139.7)
- moved C3 183.2 mm to (253.4, 156.2)
- moved C10 181.8 mm to (254.0, 162.6)
- moved J7 178.4 mm to (29.2, 167.6)
- moved U3 178.4 mm to (241.3, 156.8)
- moved U2 174.9 mm to (241.3, 141.0)
- moved C9 172.6 mm to (254.0, 146.1)
- moved J1 172.0 mm to (227.3, 153.0)
- moved C7 155.6 mm to (243.7, 76.2)
- moved L2 155.0 mm to (243.2, 69.2)
- moved C13 153.0 mm to (191.8, 148.6)
- moved U4 150.7 mm to (186.7, 149.9)
- moved C4 149.9 mm to (238.0, 72.8)
- moved L1 149.9 mm to (238.1, 67.2)
- moved D1 146.9 mm to (37.5, 167.6)
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Connections:
- J7 pad 1: Net-(D1-Pad2) -> Net-(D1-PadA)
- J8 pad 1: Net-(D2-Pad2) -> Net-(D2-PadA)
- Q2 pad 1: GND -> Net-(Q2-Pad1)
- Q2 pad 2: Net-(Q2-Pad2) -> GND
- Q2 pad 3: Net-(D1-Pad2) -> Net-(D1-PadA)
- Q3 pad 1: GND -> Net-(Q3-Pad1)
- Q3 pad 2: Net-(Q3-Pad2) -> GND
- Q3 pad 3: Net-(D2-Pad2) -> Net-(D2-PadA)
- R5 pad 1: Net-(Q2-Pad2) -> Net-(Q2-Pad1)
- R6 pad 1: Net-(Q3-Pad2) -> Net-(Q3-Pad1)
- U1 pad 11: /Resistencia_Si -> Net-(U1-Pad11)
- U1 pad 12: /Ventilador -> Net-(U1-Pad12)
- U1 pad 13: /Bomba_Agua -> Net-(U1-Pad13)
- U1 pad 14: /LEDs -> Net-(U1-Pad14)
- U1 pad 41: Net-(U1-Pad41) -> /LEDs
- U1 pad 42: Net-(U1-Pad42) -> /Bomba_Agua
- U1 pad 43: Net-(U1-Pad43) -> /Ventilador
- U1 pad 45: Net-(U1-Pad45) -> /Resistencia_Si

Commit message: Archivos KiCad
Parts:
- added D10: LED, LED_SMD:LED_0805_2012Metric, F.Cu at (44.5, 118.1)
- added D7: LED, LED_SMD:LED_0805_2012Metric, F.Cu at (45.7, 56.5)
- added D8: LED, LED_SMD:LED_0805_2012Metric, F.Cu at (34.9, 185.4)
- added D9: LED, LED_SMD:LED_0805_2012Metric, F.Cu at (77.5, 192.4)
- added J10: Test Points, Connector_PinHeader_2.54mm:PinHeader_1x07_P2.54mm_Vertical, F.Cu at (139.7, 30.5)
- added J11: JTAG Conn, Connector_PinHeader_2.54mm:PinHeader_1x05_P2.54mm_Vertical, F.Cu at (152.4, 33.0)
- added R12: 10k, Resistor_SMD:R_0805_2012Metric, F.Cu at (29.2, 175.3)
- added R13: 10k, Resistor_SMD:R_0805_2012Metric, F.Cu at (84.8, 187.3)
- added R14: 1k, Resistor_SMD:R_0805_2012Metric, F.Cu at (50.1, 56.5)
- added R15: 1k, Resistor_SMD:R_0805_2012Metric, F.Cu at (39.3, 185.4)
- added R16: 1k, Resistor_SMD:R_0805_2012Metric, F.Cu at (81.9, 192.4)
- added R17: 1k, Resistor_SMD:R_0805_2012Metric, F.Cu at (48.9, 118.1)
- added R18: 10k, Resistor_SMD:R_0805_2012Metric, F.Cu at (151.1, 189.2)
- C10, C2, C3, C9: footprint Capacitor_SMD:C_0805_2012Metric -> Capacitor_SMD:CP_Elec_4x5.8
- J7, J8: footprint MOLEX_2:MOLEX_22-29-2021 -> TerminalBlock_Phoenix:TerminalBlock_Phoenix_MKDS-1,5-2-5.08_1x02_P5.08mm_Horizontal
- R4, R7: value 1k -> 220
- R5, R6: value 1k -> 10k
- moved C10 23.4 mm to (276.9, 157.5)
- moved R5 23.4 mm to (29.2, 181.6)
- moved C9 21.3 mm to (274.3, 139.7)
- moved C3 15.8 mm to (269.1, 157.5)
- moved C2 12.0 mm to (266.0, 139.7)
Connections:
- J2 pad 29: Net-(J2-Pad29) -> /I_O_1
- J2 pad 31: Net-(J2-Pad31) -> /I_O_2
- U1 pad 18: Net-(U1-Pad18) -> /I_O_2
- U1 pad 19: Net-(U1-Pad19) -> /I_O_1

Commit message: Archivos KiCad
Parts:
- added R19: 1k, Resistor_SMD:R_0805_2012Metric, F.Cu at (66.7, -10.2)
- added R20: 1k, Resistor_SMD:R_0805_2012Metric, F.Cu at (45.7, -8.89)
- added SW1: SW_Push, Button_Switch_THT:SW_PUSH-12mm, F.Cu at (28.7, -6.09)
- added SW3: SW_Push, Button_Switch_THT:SW_PUSH-12mm, F.Cu at (67.9, -2.54)
- C1, C11, C13, C4, C5, C7: footprint Capacitor_SMD:C_0603_1608Metric -> Capacitor_SMD:C_0201_0603Metric
- C6: footprint Capacitor_SMD:C_0603_1608Metric -> Capacitor_SMD:C_0805_2012Metric
- C8: footprint Capacitor_SMD:C_0402_1005Metric -> Capacitor_SMD:C_0805_2012Metric
- D1, D2: value 1N4148W-TP -> 1N4148WS; footprint digikey-footprints:SOD-123 -> Diode_SMD:D_SOD-323
- Q2, Q3: value FMMT495TA -> MMBT2222A
- R3: footprint Resistor_SMD:R_0805_2012Metric -> Resistor_SMD:R_1206_3216Metric
- moved Q2 8.08 mm to (43.2, 172.1)
- moved D1 7.67 mm to (36.6, 175.3)
- moved D2 2.69 mm to (92.7, 178.4)
- moved Q3 1.80 mm to (92.7, 185.4)
Connections:
- J2 pad 38: Net-(J2-Pad38) -> /RPWZ_comm/Button_RPZW
- J7 pad 1: Net-(D1-PadA) -> Net-(D1-Pad2)
- J8 pad 1: Net-(D2-PadA) -> Net-(D2-Pad2)
- Q2 pad 3: Net-(D1-PadA) -> Net-(D1-Pad2)
- Q3 pad 3: Net-(D2-PadA) -> Net-(D2-Pad2)
- U1 pad 25: Net-(U1-Pad25) -> /STM32/Button_STM32

Commit message: Archivos KiCad
Parts:
- added J12: Conn_USART, TerminalBlock_Phoenix:TerminalBlock_Phoenix_MKDS-1,5-2-5.08_1x02_P5.08mm_Horizontal, F.Cu at (125.7, 31.1)
- C1, C11, C13, C4, C5, C7: footprint Capacitor_SMD:C_0201_0603Metric -> Capacitor_SMD:C_0805_2012Metric
- moved J1 114.2 mm to (114.9, 132.7)
- moved J5 96.5 mm to (88.3, 127.0)
- moved J6 78.3 mm to (91.4, 109.9), turned to 270 degrees
Connections:
- U1 pad 12: Net-(U1-Pad12) -> /STM32/TX2
- U1 pad 13: Net-(U1-Pad13) -> /STM32/RX2

Commit message: Archivos KiCad
Parts:
- added H2: MountingHole, MountingHole:MountingHole_3.5mm, F.Cu at (182.5, 83.5)
- added H3: MountingHole, MountingHole:MountingHole_3.5mm, F.Cu at (105.0, 120.0)
- C2, C3: footprint Capacitor_SMD:CP_Elec_4x5.8 -> Capacitor_SMD:CP_Elec_6.3x5.9
- D10: value LED -> LEDs
- D3: value LED -> LED_5V
- D4: value LED -> LED_3.3V
- D5: value LED -> LED_STM
- D6: value LED -> LED_RPZW
- D7: value LED -> LED_RSi
- D8: value LED -> LED_Vent
- D9: value LED -> LED_H2O
- J12: footprint TerminalBlock_Phoenix:TerminalBlock_Phoenix_MKDS-1,5-2-5.08_1x02_P5.08mm_Horizontal -> Connector_PinHeader_2.54mm:PinHeader_1x02_P2.54mm_Vertical
- SW1, SW3: footprint Button_Switch_THT:SW_PUSH-12mm -> Button_Switch_THT:SW_PUSH_6mm_H4.3mm
- moved SW1 147.8 mm to (138.7, 92.7)
- moved R20 145.9 mm to (138.7, 103.5), turned to 90 degrees
- moved Q1 136.6 mm to (162.8, 82.3), turned to 90 degrees
- moved R19 133.0 mm to (113.3, 114.5), turned to 270 degrees
- moved C10 127.0 mm to (160.3, 107.2)
- moved L2 124.7 mm to (128.0, 116.8)
- moved SW3 124.5 mm to (116.1, 112.3)
- moved J7 123.6 mm to (118.6, 82.2), turned to 180 degrees
- moved R5 123.0 mm to (115.3, 93.7), turned to 180 degrees
- moved R4 121.7 mm to (153.2, 106.9), turned to 270 degrees
- moved R12 121.5 mm to (119.3, 93.7), turned to 180 degrees
- moved R3 120.7 mm to (154.7, 89.2), turned to 180 degrees
- moved L1 120.2 mm to (128.0, 115.6), turned to 180 degrees
- moved D1 116.3 mm to (115.8, 90.2)
- moved R11 114.6 mm to (118.1, 125.1), turned to 270 degrees
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Connections:
- J5 pad 1: /In_Out/120VAC -> GNDREF
- J5 pad 2: GNDREF -> /In_Out/120VAC
- J6 pad 1: Net-(J6-Pad1) -> /In_Out/120VAC
- J6 pad 2: /In_Out/120VAC -> Net-(J6-Pad2)
- Q1 pad 2: Net-(J6-Pad1) -> Net-(J6-Pad2)
- R3 pad 1: Net-(J6-Pad1) -> Net-(J6-Pad2)
Routing:
- net +12V: track 0.00 -> 116.3 mm
- net Net-(J6-Pad2): track 0.00 -> 30.0 mm
- net /DHT22: track 0.00 -> 11.5 mm
- net Net-(J9-Pad1): track 0.00 -> 11.2 mm
- net +3V3: track 0.00 -> 11.1 mm
- net /STM32/VDDA: track 0.00 -> 10.7 mm
- net +5V: track 0.00 -> 7.81 mm
- net GND: track 0.00 -> 7.69 mm
- net /In_Out/120VAC: track 0.00 -> 7.62 mm
- net GNDREF: track 0.00 -> 7.57 mm
- net Net-(L1-Pad1): track 0.00 -> 5.80 mm
- net Net-(D8-Pad2): track 0.00 -> 3.92 mm
- net Net-(D9-Pad2): track 0.00 -> 3.81 mm
- net Net-(D7-Pad2): track 0.00 -> 3.76 mm
- net Net-(D10-Pad2): track 0.00 -> 3.74 mm
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Other:
- board size 105.4 x 72.4 mm -> 108 x 57.5 mm

Commit message: Archivos KiCad
Parts:
- removed ? (x4): , RPi_Hat:RPi_Hat_Mounting_Hole
- removed the R11 at (118.1, 125.1)
- removed R19: 1k, Resistor_SMD:R_0805_2012Metric
- removed SW3: SW_Push, Button_Switch_THT:SW_PUSH_6mm_H4.3mm
- added J13: RPZW_RST, Connector_PinHeader_2.54mm:PinHeader_1x02_P2.54mm_Vertical, F.Cu at (132.6, 125.3)
- added R10: 1k, Resistor_SMD:R_0805_2012Metric, F.Cu at (191.9, 96.0)
- added SW2: RPZW_RST_Push, Button_Switch_THT:SW_PUSH_6mm_H4.3mm, F.Cu at (91.7, 118.3)
- D1, D2: value 1N4148WS -> MRA4004T3G; footprint Diode_SMD:D_SOD-323 -> Diode_SMD:D_SMA
- J12: value Conn_USART -> USART_Conn; footprint Connector_PinHeader_2.54mm:PinHeader_1x02_P2.54mm_Vertical -> Connector_PinHeader_2.54mm:PinHeader_1x03_P2.54mm_Vertical
- moved J10 94.2 mm to (104.5, 130.1), turned to 90 degrees
- moved J11 94.1 mm to (108.5, 125.2), turned to 90 degrees
- moved D10 92.3 mm to (195.6, 123.5), turned to 180 degrees
- moved D8 90.0 mm to (195.6, 112.5), turned to 180 degrees
- moved R17 88.3 mm to (191.9, 123.5), turned to 0 degrees
- moved D9 85.6 mm to (195.6, 118.0), turned to 180 degrees
- moved R15 85.1 mm to (191.9, 112.5), turned to 0 degrees
- moved D5 84.9 mm to (195.6, 96.0), turned to 180 degrees
- moved D7 84.5 mm to (195.6, 107.0), turned to 180 degrees
- moved R16 81.2 mm to (191.9, 118.0), turned to 0 degrees
- moved D6 79.5 mm to (195.6, 101.5), turned to 180 degrees
- moved R14 79.4 mm to (191.9, 107.0), turned to 0 degrees
- moved R11 74.1 mm to (191.9, 101.5), turned to 0 degrees
- moved SW1 36.2 mm to (106.6, 109.5)
- moved R20 24.6 mm to (116.0, 113.0), turned to 270 degrees
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- renumbered R10 to R11
Connections:
- net Net-(L1-Pad1) renamed /STM32/VSSA
- J12 pad 1: /STM32/TX2 -> GND
- U1 pad 10: Net-(U1-Pad10) -> /Resistencia_Si
- U1 pad 11: Net-(U1-Pad11) -> /Bomba_Agua
- U1 pad 12: /STM32/TX2 -> /Ventilador
- U1 pad 13: /STM32/RX2 -> /LEDs
- U1 pad 15: /LM35 -> /DHT22
- U1 pad 17: /DHT22 -> /LM35
- U1 pad 21: /SCL_I2C -> /STM32/TX2
- U1 pad 22: /SDA_I2C -> /STM32/RX2
- U1 pad 25: /STM32/Button_STM32 -> Net-(U1-Pad25)
- U1 pad 41: /LEDs -> Net-(U1-Pad41)
- U1 pad 42: /Bomba_Agua -> /SCL_I2C
- U1 pad 43: /Ventilador -> /SDA_I2C
- U1 pad 45: /Resistencia_Si -> Net-(U1-Pad45)
Routing:
- net +5V: track 7.81 -> 38.8 mm
- net Net-(J6-Pad2): track 30.0 -> 44.7 mm
- net Net-(R7-Pad1): track 0.00 -> 13.2 mm
- net Net-(D2-Pad2): track 0.00 -> 12.3 mm
- net Net-(D1-Pad2): track 0.00 -> 12.0 mm
- net /STM32/VDDA: track 10.7 -> 0.00 mm
- net Net-(Q1-Pad3): track 0.00 -> 10.5 mm
- net GND: track 7.69 -> 1.70 mm
- net /STM32/VSSA: track 5.80 -> 0.00 mm
- net Net-(Q3-Pad1): track 0.00 -> 5.73 mm
- net Net-(Q2-Pad1): track 0.00 -> 4.66 mm
- net Net-(D8-Pad2): track 3.92 -> 0.00 mm
- net Net-(D9-Pad2): track 3.81 -> 0.00 mm
- net Net-(D7-Pad2): track 3.76 -> 0.00 mm
- net Net-(D10-Pad2): track 3.74 -> 0.00 mm
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
Commit message: Archivos KiCad
Parts:
- removed J11: JTAG Conn, Connector_PinHeader_2.54mm:PinHeader_1x05_P2.54mm_Vertical
- moved U4 41.2 mm to (123.9, 110.2), turned to 90 degrees
- moved C13 29.4 mm to (129.1, 111.4), turned to 90 degrees
- moved L1 1.79 mm to (140.8, 102.9), turned to 0 degrees
- moved L2 0.91 mm to (139.1, 104.1), turned to 180 degrees
Connections:
- J2 pad 11: Net-(J2-Pad11) -> /JNTRST
- J2 pad 13: /JTMS -> Net-(J2-Pad13)
- J2 pad 15: /JNTRST -> /JTDO
- J2 pad 18: /JTDO -> Net-(J2-Pad18)
- J2 pad 19: Net-(J2-Pad19) -> /JTDI
- J2 pad 21: Net-(J2-Pad21) -> /JTCK
- J2 pad 22: /JTCK -> Net-(J2-Pad22)
- J2 pad 23: Net-(J2-Pad23) -> /JTMS
- J2 pad 37: /JTDI -> Net-(J2-Pad37)
Routing:
- net +5V: track 38.8 -> 280.2 mm, vias 0 -> 7
- net +3V3: track 12.3 -> 214.5 mm, vias 0 -> 4
- net Net-(J2-Pad40): track 0.00 -> 114.1 mm, vias 0 -> 2
- net /Ventilador: track 0.00 -> 110.1 mm, vias 0 -> 2
- net /LEDs: track 0.07 -> 99.7 mm, vias 0 -> 2
- net /Bomba_Agua: track 0.00 -> 91.2 mm, vias 0 -> 2
- net +12V: track 119.2 -> 203.8 mm, vias 0 -> 2
- net /Resistencia_Si: track 0.00 -> 71.3 mm, vias 0 -> 2
- net /HD38: track 0.00 -> 62.9 mm, vias 0 -> 2
- net /DHT22: track 15.2 -> 77.3 mm, vias 0 -> 2
- net Net-(R10-Pad1): track 0.00 -> 55.4 mm, vias 0 -> 2
- net Net-(J13-Pad2): track 0.00 -> 48.2 mm
- net /USART1: track 0.00 -> 44.3 mm, vias 0 -> 1
- net /RPWZ_comm/Button_RPZW: track 0.00 -> 43.6 mm
- net /USART2: track 0.00 -> 43.4 mm, vias 0 -> 1
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