File: RPi_Zero_pHat_Template-master/RPi_Zero_pHat_Template.kicad_pcb (KiCad board)
At the start: 2 copper layers, 108 x 57.5 mm, 69 parts, among them J1 POWER_JACK, J10 Test Points, J12 USART_Conn, J13 RPZW_RST, J2 RPi_GPIO, J3 DHT22 Conn, J4 HD38 Conn, J5 120VAC, J6 R_Si, J7 Ventilador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

Commit message: Archivos KiCad
Routing:
- net +5V: track 280.2 -> 292.6 mm
- net /Ventilador: track 110.1 -> 104.0 mm
- net +12V: track 203.8 -> 205.5 mm
- net /Bomba_Agua: track 91.2 -> 90.1 mm
- net +3V3: track 214.5 -> 213.5 mm
- net Net-(R10-Pad1): track 55.4 -> 56.0 mm
Other:
- net class Default: trace_width 0.25 -> 0.2; via_drill 0.4 -> 0.2
- rule via_min_drill: 0.3 -> 0.2

Commit message: Archivos KiCad
Routing:
- net +5V: track 292.6 -> 288.3 mm, vias 7 -> 5
