File: RPi_Zero_pHat_Template-master/RPi_Zero_pHat_Template.kicad_pcb (KiCad board)
At the start: 2 copper layers, 108 x 57.5 mm, 69 parts, among them J1 POWER_JACK, J10 Test Points, J12 USART_Conn, J13 RPZW_RST, J2 RPi_GPIO, J3 DHT22 Conn, J4 HD38 Conn, J5 120VAC, J6 R_Si, J7 Ventilador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

Commit message: Archivos KiCad
Parts:
- removed C13: 100nF, Capacitor_SMD:C_0805_2012Metric
- removed U4: LM35, digikey-footprints:SOIC-8_W3.9mm
- C10, C9: footprint Capacitor_SMD:CP_Elec_4x5.8 -> Capacitor_SMD:CP_Elec_3x5.4
- C2, C3: footprint Capacitor_SMD:CP_Elec_6.3x5.9 -> Capacitor_SMD:CP_Elec_4x5.8
- J10: footprint Connector_PinHeader_2.54mm:PinHeader_1x07_P2.54mm_Vertical -> Connector_PinHeader_2.54mm:PinHeader_1x06_P2.54mm_Vertical
- J3, J4: footprint RJ9-Conn:520249-2 -> RJ9-Conn:RJ9-4P4C
- L1, L2: footprint Inductor_SMD:L_0402_1005Metric -> Inductor_SMD:L_0603_1608Metric
- moved J3 3.61 mm to (94.7, 94.2)
- moved J4 3.02 mm to (94.7, 109.3)
- moved J1 1.92 mm to (173.7, 72.5)
- moved R18 1.52 mm to (99.7, 102.1)
- moved L1 0.98 mm to (139.9, 102.7)
- moved L2 0.85 mm to (139.8, 104.5)
- renumbered J13 to J11, R20 to R19
Connections:
- J10 pad 5: /LM35 -> /HD38
- J10 pad 6: /HD38 -> /DHT22
- U1 pad 17: /LM35 -> Net-(U1-Pad17)
Routing:
- net /LM35: track 37.2 -> 0.00 mm, vias 2 -> 0
- net +5V: track 288.3 -> 253.8 mm, vias 5 -> 3
- net GND: track 5.34 -> 0.93 mm
- net /Resistencia_Si: track 71.3 -> 73.3 mm
- net /DHT22: track 77.2 -> 75.3 mm
- net +3V3: track 214.1 -> 213.0 mm
- net /HD38: track 62.9 -> 62.1 mm
- net +12V: track 205.5 -> 204.8 mm
- net /STM32/VSSA: track 7.06 -> 6.44 mm
- net /STM32/VDDA: track 8.98 -> 9.60 mm

Commit message: Archivos KiCad
Parts:
- added H4: MountingHole, MountingHole:MountingHole_3.5mm, F.Cu at (182.5, 122.5)
- moved H2 2.50 mm to (182.5, 86.0)
- moved H3 2.50 mm to (105.0, 122.5)
Routing:
- net +3V3: track 213.0 -> 267.1 mm, vias 4 -> 7
- net +5V: track 253.8 -> 284.6 mm, vias 3 -> 4
- net +12V: track 204.8 -> 200.1 mm, vias 2 -> 0
- net /LEDs: track 99.7 -> 98.0 mm
- net Net-(J11-Pad1): track 41.9 -> 43.1 mm
- net Net-(J11-Pad2): track 48.2 -> 47.2 mm
- net /DHT22: track 75.3 -> 75.4 mm, vias 2 -> 1
- net /HD38: track 62.1 -> 62.2 mm, vias 2 -> 1
- net Net-(J2-Pad40): vias 2 -> 1

Commit message: Archivos KiCad
Parts:
- removed H4: MountingHole, MountingHole:MountingHole_3.5mm
- added ?: , RPi_Hat:RPi_Hat_Mounting_Hole, F.Cu at (185.8, 106.1)
- added ?: , RPi_Hat:RPi_Hat_Mounting_Hole, F.Cu at (127.8, 129.1)
- moved C2 2.44 mm to (178.6, 108.6)
Routing:
- net GND: track 0.93 -> 54.8 mm, vias 0 -> 11
- net (no net): track 0.00 -> 5.70 mm, vias 0 -> 4
- net Net-(J2-Pad40): track 114.4 -> 111.5 mm
- net /Resistencia_Si: track 73.3 -> 75.6 mm
- net +12V: track 200.1 -> 201.4 mm
- net Net-(J11-Pad1): track 43.1 -> 44.3 mm
- net +3V3: track 267.1 -> 266.2 mm
- added copper zone on B.Cu, net GND
- added copper zone on F.Cu, net GND

Commit message: Archivos KiCad
Routing:
- net GND: track 54.8 -> 109.2 mm, vias 11 -> 63
- net (no net): track 5.70 -> 0.00 mm, vias 4 -> 0
