File: RPi_Zero_pHat_Template-master/Alimentacion.sch (KiCad schematic (older format))
At the start: 16 parts, among them J1 POWER_JACK, U2 V7805-1000, U3 V7803-1000

Commit message: Archivos KiCad
Parts:
- removed C1, C11, C4, C7, C8: 100nF, Capacitor_SMD:C_0805_2012Metric, symbol Device:C
- removed C12: 4.7uF, Capacitor_SMD:C_0805_2012Metric, symbol Device:C
- removed C5: 10nF, Capacitor_SMD:C_0805_2012Metric, symbol Device:C
- removed C6: 1uF, Capacitor_SMD:C_0805_2012Metric, symbol Device:C
- removed L2: L, Inductor_SMD:L_0805_2012Metric, symbol Device:L
Other:
- moved on the sheet: C10, C2, C3, C9, J1, U2, U3

Commit message: Archivos KiCad
Parts:
- added D3, D4: LED, LED_SMD:LED_0805_2012Metric, symbol Device:LED
- added R8, R9: 1k, Resistor_SMD:R_0805_2012Metric, symbol Device:R
Connections:
- net +3V3: now also R9.2
- net +5V: now also R8.2
- net GND: now also D3.1 (K), D4.1 (K)
- new net: D3.2 (A), R8.1
- new net: D4.2 (A), R9.1
Changed lines of the file:
@@
 L power:+5V #PWR?
 U 1 1 607E7D05
-P 5650 3100
+P 6250 3100
 AR Path="/607E7D05" Ref="#PWR?"  Part="1"
 AR Path="/607B7D6E/607E7D05" Ref="#PWR0116"  Part="1"
-F 0 "#PWR0116" H 5650 2950 50  0001 C CNN
-F 1 "+5V" V 5665 3228 50  0000 L CNN
-F 2 "" H 5650 3100 50  0001 C CNN
-F 3 "" H 5650 3100 50  0001 C CNN
-	1    5650 3100
+F 0 "#PWR0116" H 6250 2950 50  0001 C CNN
+F 1 "+5V" V 6265 3228 50  0000 L CNN
+F 2 "" H 6250 3100 50  0001 C CNN
+F 3 "" H 6250 3100 50  0001 C CNN
+	1    6250 3100
 	0    1    1    0
 $EndComp
-Wire Wire Line
-	5650 3100 5500 3100
 Connection ~ 5500 3100
 $Comp
@@
 Wire Wire Line
 	5500 4250 5500 4350
-Wire Wire Line
-	5650 4250 5500 4250
 Connection ~ 5500 4250
 Wire Wire Line
@@
 L power:+3.3V #PWR?
 U 1 1 607E7D5F
-P 5650 4250
+P 6250 4250
 AR Path="/607E7D5F" Ref="#PWR?"  Part="1"
 AR Path="/607B7D6E/607E7D5F" Ref="#PWR0124"  Part="1"
-F 0 "#PWR0124" H 5650 4100 50  0001 C CNN
-F 1 "+3.3V" V 5665 4378 50  0000 L CNN
-F 2 "" H 5650 4250 50  0001 C CNN
-F 3 "" H 5650 4250 50  0001 C CNN
-	1    5650 4250
+F 0 "#PWR0124" H 6250 4100 50  0001 C CNN
+F 1 "+3.3V" V 6265 4378 50  0000 L CNN
+F 2 "" H 6250 4250 50  0001 C CNN
+F 3 "" H 6250 4250 50  0001 C CNN
+	1    6250 4250
 	0    1    1    0
 $EndComp
@@
 	0    -1   -1   0
 $EndComp
+$Comp
+L Device:R R?
+U 1 1 6078B5B7
+P 6000 3300
+AR Path="/6081C49D/6078B5B7" Ref="R?"  Part="1"
+AR Path="/607B7D6E/6078B5B7" Ref="R8"  Part="1"
+F 0 "R8" V 5793 3300 50  0000 C CNN
+F 1 "1k" V 5884 3300 50  0000 C CNN
+F 2 "Resistor_SMD:R_0805_2012Metric" V 5930 3300 50  0001 C CNN
+F 3 "~" H 6000 3300 50  0001 C CNN
+	1    6000 3300
+	-1   0    0    1
+$EndComp
+Wire Wire Line
+	5500 3100 6000 3100
+Wire Wire Line
+	5500 4250 6000 4250
+Wire Wire Line
+	6000 3150 6000 3100
+Connection ~ 6000 3100
+Wire Wire Line
+	6000 3100 6250 3100
+$Comp
+L Device:R R?
+U 1 1 6078C3C2
+P 6000 4450
+AR Path="/6081C49D/6078C3C2" Ref="R?"  Part="1"
+AR Path="/607B7D6E/6078C3C2" Ref="R9"  Part="1"
+F 0 "R9" V 5793 4450 50  0000 C CNN
+F 1 "1k" V 5884 4450 50  0000 C CNN
+F 2 "Resistor_SMD:R_0805_2012Metric" V 5930 4450 50  0001 C CNN
+F 3 "~" H 6000 4450 50  0001 C CNN
+	1    6000 4450
+	-1   0    0    1
+$EndComp
+Wire Wire Line
+	6000 4300 6000 4250
+Connection ~ 6000 4250
+Wire Wire Line
+	6000 4250 6250 4250
+$Comp
+L Device:LED D3
+U 1 1 6078CF49
+P 6200 3450
+F 0 "D3" H 6200 3700 50  0000 C CNN
+F 1 "LED" H 6200 3600 50  0000 C CNN
+F 2 "LED_SMD:LED_0805_2012Metric" H 6200 3450 50  0001 C CNN
+F 3 "~" H 6200 3450 50  0001 C CNN
+	1    6200 3450
+	-1   0    0    1
+$EndComp
+$Comp
+L Device:LED D4
+U 1 1 6078E428
+P 6200 4600
+F 0 "D4" H 6200 4850 50  0000 C CNN
+F 1 "LED" H 6200 4750 50  0000 C CNN
+F 2 "LED_SMD:LED_0805_2012Metric" H 6200 4600 50  0001 C CNN
+F 3 "~" H 6200 4600 50  0001 C CNN
+	1    6200 4600
+	-1   0    0    1
+$EndComp
+Wire Wire Line
+	6050 3450 6000 3450
+Wire Wire Line
+	6050 4600 6000 4600
+$Comp
+L power:GND #PWR?
+U 1 1 6078F355
+P 6400 4650
+AR Path="/6078F355" Ref="#PWR?"  Part="1"
+AR Path="/607B7D6E/6078F355" Ref="#PWR0146"  Part="1"
+F 0 "#PWR0146" H 6400 4400 50  0001 C CNN
+F 1 "GND" H 6405 4477 50  0000 C CNN
+F 2 "" H 6400 4650 50  0001 C CNN
+F 3 "" H 6400 4650 50  0001 C CNN
+	1    6400 4650
+	1    0    0    -1
+$EndComp
+Wire Wire Line
+	6400 3500 6400 3450
+Wire Wire Line
+	6400 3450 6350 3450
+Wire Wire Line
+	6350 4600 6400 4600
+Wire Wire Line
+	6400 4600 6400 4650
+$Comp
+L power:GND #PWR?
+U 1 1 60790675
+P 6400 3500
+AR Path="/60790675" Ref="#PWR?"  Part="1"
+AR Path="/607B7D6E/60790675" Ref="#PWR0147"  Part="1"
+F 0 "#PWR0147" H 6400 3250 50  0001 C CNN
+F 1 "GND" H 6405 3327 50  0000 C CNN
+F 2 "" H 6400 3500 50  0001 C CNN
+F 3 "" H 6400 3500 50  0001 C CNN
+	1    6400 3500
+	1    0    0    -1
+$EndComp
 $EndSCHEMATC

Commit message: Archivos KiCad
Parts:
- removed C10, C9: 22uF, Capacitor_SMD:C_0805_2012Metric, symbol Device:C
- removed C2, C3: 10uF, Capacitor_SMD:C_0805_2012Metric, symbol Device:C
- added C10, C9: 22uF, Capacitor_SMD:CP_Elec_4x5.8, symbol Device:CP
- added C2, C3: 10uF, Capacitor_SMD:CP_Elec_4x5.8, symbol Device:CP
Connections:
- net +12V: now also C2.1
- net +3V3: now also C10.1
- net +5V: now also C3.1, C9.1
- net GND: now also C10.2, C2.2, C3.2, C9.2
Changed lines of the file:
@@
-$EndComp
-$Comp
-L Device:C C?
-U 1 1 607E7CE9
-P 4400 3350
-AR Path="/607E7CE9" Ref="C?"  Part="1"
-AR Path="/607B7D6E/607E7CE9" Ref="C2"  Part="1"
-F 0 "C2" H 4515 3396 50  0000 L CNN
-F 1 "10uF" H 4515 3305 50  0000 L CNN
-F 2 "Capacitor_SMD:C_0805_2012Metric" H 4438 3200 50  0001 C CNN
-F 3 "~" H 4400 3350 50  0001 C CNN
-	1    4400 3350
-	1    0    0    -1
-$EndComp
-$Comp
-L Device:C C?
-U 1 1 607E7CEF
-P 5500 3350
-AR Path="/607E7CEF" Ref="C?"  Part="1"
-AR Path="/607B7D6E/607E7CEF" Ref="C9"  Part="1"
-F 0 "C9" H 5615 3396 50  0000 L CNN
-F 1 "22uF" H 5615 3305 50  0000 L CNN
-F 2 "Capacitor_SMD:C_0805_2012Metric" H 5538 3200 50  0001 C CNN
-F 3 "~" H 5500 3350 50  0001 C CNN
-	1    5500 3350
-	1    0    0    -1
 $EndComp
 $Comp
@@
 $EndComp
 $Comp
-L Device:C C?
-U 1 1 607E7D39
-P 4400 4500
-AR Path="/607E7D39" Ref="C?"  Part="1"
-AR Path="/607B7D6E/607E7D39" Ref="C3"  Part="1"
-F 0 "C3" H 4515 4546 50  0000 L CNN
-F 1 "10uF" H 4515 4455 50  0000 L CNN
-F 2 "Capacitor_SMD:C_0805_2012Metric" H 4438 4350 50  0001 C CNN
-F 3 "~" H 4400 4500 50  0001 C CNN
-	1    4400 4500
-	1    0    0    -1
-$EndComp
-$Comp
-L Device:C C?
-U 1 1 607E7D3F
-P 5500 4500
-AR Path="/607E7D3F" Ref="C?"  Part="1"
-AR Path="/607B7D6E/607E7D3F" Ref="C10"  Part="1"
-F 0 "C10" H 5615 4546 50  0000 L CNN
-F 1 "22uF" H 5615 4455 50  0000 L CNN
-F 2 "Capacitor_SMD:C_0805_2012Metric" H 5538 4350 50  0001 C CNN
-F 3 "~" H 5500 4500 50  0001 C CNN
-	1    5500 4500
-	1    0    0    -1
-$EndComp
-$Comp
 L power:GND #PWR?
 U 1 1 607E7D45
@@
 	1    0    0    -1
 $EndComp
+$Comp
+L Device:CP C3
+U 1 1 607F0080
+P 4400 4500
+F 0 "C3" H 4518 4546 50  0000 L CNN
+F 1 "10uF" H 4518 4455 50  0000 L CNN
+F 2 "Capacitor_SMD:CP_Elec_4x5.8" H 4438 4350 50  0001 C CNN
+F 3 "~" H 4400 4500 50  0001 C CNN
+	1    4400 4500
+	1    0    0    -1
+$EndComp
+$Comp
+L Device:CP C9
+U 1 1 607F08D8
+P 5500 3350
+F 0 "C9" H 5618 3396 50  0000 L CNN
+F 1 "22uF" H 5618 3305 50  0000 L CNN
+F 2 "Capacitor_SMD:CP_Elec_4x5.8" H 5538 3200 50  0001 C CNN
+F 3 "~" H 5500 3350 50  0001 C CNN
+	1    5500 3350
+	1    0    0    -1
+$EndComp
+$Comp
+L Device:CP C2
+U 1 1 607F15B9
+P 4400 3350
+F 0 "C2" H 4518 3396 50  0000 L CNN
+F 1 "10uF" H 4518 3305 50  0000 L CNN
+F 2 "Capacitor_SMD:CP_Elec_4x5.8" H 4438 3200 50  0001 C CNN
+F 3 "~" H 4400 3350 50  0001 C CNN
+	1    4400 3350
+	1    0    0    -1
+$EndComp
+$Comp
+L Device:CP C10
+U 1 1 607F2EF9
+P 5500 4500
+F 0 "C10" H 5618 4546 50  0000 L CNN
+F 1 "22uF" H 5618 4455 50  0000 L CNN
+F 2 "Capacitor_SMD:CP_Elec_4x5.8" H 5538 4350 50  0001 C CNN
+F 3 "~" H 5500 4500 50  0001 C CNN
+	1    5500 4500
+	1    0    0    -1
+$EndComp

Commit message: Archivos KiCad
Parts:
- C2, C3: footprint Capacitor_SMD:CP_Elec_4x5.8 -> Capacitor_SMD:CP_Elec_6.3x5.9
- D3: value LED -> LED_5V
- D4: value LED -> LED_3.3V
Changed lines of the file:
@@
 P 6200 3450
 F 0 "D3" H 6200 3700 50  0000 C CNN
-F 1 "LED" H 6200 3600 50  0000 C CNN
+F 1 "LED_5V" H 6200 3600 50  0000 C CNN
 F 2 "LED_SMD:LED_0805_2012Metric" H 6200 3450 50  0001 C CNN
 F 3 "~" H 6200 3450 50  0001 C CNN
@@
 P 6200 4600
 F 0 "D4" H 6200 4850 50  0000 C CNN
-F 1 "LED" H 6200 4750 50  0000 C CNN
+F 1 "LED_3.3V" H 6200 4750 50  0000 C CNN
 F 2 "LED_SMD:LED_0805_2012Metric" H 6200 4600 50  0001 C CNN
 F 3 "~" H 6200 4600 50  0001 C CNN
@@
 F 0 "C3" H 4518 4546 50  0000 L CNN
 F 1 "10uF" H 4518 4455 50  0000 L CNN
-F 2 "Capacitor_SMD:CP_Elec_4x5.8" H 4438 4350 50  0001 C CNN
+F 2 "Capacitor_SMD:CP_Elec_6.3x5.9" H 4438 4350 50  0001 C CNN
 F 3 "~" H 4400 4500 50  0001 C CNN
 	1    4400 4500
@@
 F 0 "C2" H 4518 3396 50  0000 L CNN
 F 1 "10uF" H 4518 3305 50  0000 L CNN
-F 2 "Capacitor_SMD:CP_Elec_4x5.8" H 4438 3200 50  0001 C CNN
+F 2 "Capacitor_SMD:CP_Elec_6.3x5.9" H 4438 3200 50  0001 C CNN
 F 3 "~" H 4400 3350 50  0001 C CNN
 	1    4400 3350

Commit message: Archivos KiCad
Parts:
- C10, C9: footprint Capacitor_SMD:CP_Elec_4x5.8 -> Capacitor_SMD:CP_Elec_3x5.4
- C2, C3: footprint Capacitor_SMD:CP_Elec_6.3x5.9 -> Capacitor_SMD:CP_Elec_4x5.8
Changed lines of the file:
@@
 F 0 "C3" H 4518 4546 50  0000 L CNN
 F 1 "10uF" H 4518 4455 50  0000 L CNN
-F 2 "Capacitor_SMD:CP_Elec_6.3x5.9" H 4438 4350 50  0001 C CNN
+F 2 "Capacitor_SMD:CP_Elec_4x5.8" H 4438 4350 50  0001 C CNN
 F 3 "~" H 4400 4500 50  0001 C CNN
 	1    4400 4500
@@
 F 0 "C9" H 5618 3396 50  0000 L CNN
 F 1 "22uF" H 5618 3305 50  0000 L CNN
-F 2 "Capacitor_SMD:CP_Elec_4x5.8" H 5538 3200 50  0001 C CNN
+F 2 "Capacitor_SMD:CP_Elec_3x5.4" H 5538 3200 50  0001 C CNN
 F 3 "~" H 5500 3350 50  0001 C CNN
 	1    5500 3350
@@
 F 0 "C2" H 4518 3396 50  0000 L CNN
 F 1 "10uF" H 4518 3305 50  0000 L CNN
-F 2 "Capacitor_SMD:CP_Elec_6.3x5.9" H 4438 3200 50  0001 C CNN
+F 2 "Capacitor_SMD:CP_Elec_4x5.8" H 4438 3200 50  0001 C CNN
 F 3 "~" H 4400 3350 50  0001 C CNN
 	1    4400 3350
@@
 F 0 "C10" H 5618 4546 50  0000 L CNN
 F 1 "22uF" H 5618 4455 50  0000 L CNN
-F 2 "Capacitor_SMD:CP_Elec_4x5.8" H 5538 4350 50  0001 C CNN
+F 2 "Capacitor_SMD:CP_Elec_3x5.4" H 5538 4350 50  0001 C CNN
 F 3 "~" H 5500 4500 50  0001 C CNN
 	1    5500 4500
