File: RPi_Zero_pHat_Template-master/RPWZ_comm.sch (KiCad schematic (older format))
At the start: 1 part, among them J2 RPi_GPIO

Commit message: Archivos KiCad
Parts:
- added D6: LED, LED_SMD:LED_0805_2012Metric, symbol Device:LED
- added R10: 1k, Resistor_SMD:R_0805_2012Metric, symbol Device:R
Connections:
- net GND: now also D6.1 (K)
- net at J2.40 (GPIO21): now also R10.1
- new net: D6.2 (A), R10.2
Changed lines of the file:
@@
 Text HLabel 6300 4100 2    50   Input ~ 0
 RPWZ_BOOT
+$Comp
+L Device:R R?
+U 1 1 607E2837
+P 6150 4800
+AR Path="/6081C49D/607E2837" Ref="R?"  Part="1"
+AR Path="/607B7D6E/607E2837" Ref="R?"  Part="1"
+AR Path="/60760232/607E2837" Ref="R?"  Part="1"
+AR Path="/60805E76/607E2837" Ref="R10"  Part="1"
+F 0 "R10" V 5943 4800 50  0000 C CNN
+F 1 "1k" V 6034 4800 50  0000 C CNN
+F 2 "Resistor_SMD:R_0805_2012Metric" V 6080 4800 50  0001 C CNN
+F 3 "~" H 6150 4800 50  0001 C CNN
+	1    6150 4800
+	1    0    0    -1
+$EndComp
+$Comp
+L Device:LED D?
+U 1 1 607E283D
+P 6150 5100
+AR Path="/607B7D6E/607E283D" Ref="D?"  Part="1"
+AR Path="/60760232/607E283D" Ref="D?"  Part="1"
+AR Path="/60805E76/607E283D" Ref="D6"  Part="1"
+F 0 "D6" H 6150 5350 50  0000 C CNN
+F 1 "LED" H 6150 5250 50  0000 C CNN
+F 2 "LED_SMD:LED_0805_2012Metric" H 6150 5100 50  0001 C CNN
+F 3 "~" H 6150 5100 50  0001 C CNN
+	1    6150 5100
+	0    -1   -1   0
+$EndComp
+Wire Wire Line
+	6150 5300 6150 5250
+$Comp
+L power:GND #PWR?
+U 1 1 607E2844
+P 6150 5300
+AR Path="/607E2844" Ref="#PWR?"  Part="1"
+AR Path="/607B7D6E/607E2844" Ref="#PWR?"  Part="1"
+AR Path="/60760232/607E2844" Ref="#PWR?"  Part="1"
+AR Path="/60805E76/607E2844" Ref="#PWR0149"  Part="1"
+F 0 "#PWR0149" H 6150 5050 50  0001 C CNN
+F 1 "GND" H 6155 5127 50  0000 C CNN
+F 2 "" H 6150 5300 50  0001 C CNN
+F 3 "" H 6150 5300 50  0001 C CNN
+	1    6150 5300
+	1    0    0    -1
+$EndComp
+Wire Wire Line
+	6150 4500 6000 4500
+Wire Wire Line
+	6150 4500 6150 4650
 $EndSCHEMATC

Commit message: Archivos KiCad
Connections:
- net RPZW_IO2: now reaches J2.29 (GPIO05)
- net RPZW_IO1: now reaches J2.31 (GPIO06)
Changed lines of the file:
@@
 Wire Wire Line
 	6150 4500 6150 4650
+Wire Wire Line
+	4100 4000 3800 4000
+Wire Wire Line
+	4100 4100 3800 4100
+Text HLabel 3800 4100 0    50   Input ~ 0
+RPZW_IO1
+Text HLabel 3800 4000 0    50   Input ~ 0
+RPZW_IO2
 $EndSCHEMATC

Commit message: Archivos KiCad
Parts:
- added R20: 1k, Resistor_SMD:R_0805_2012Metric, symbol Device:R
- added SW1: SW_Push, Button_Switch_THT:SW_PUSH-12mm, symbol Switch:SW_Push
Connections:
- net GND: now also R20.1
- net Button_RPZW: now reaches J2.38 (GPIO20)
- net Button_RPZW: now also R20.2, SW1.2
- new net +3V3: SW1.1
Changed lines of the file:
@@
 Text HLabel 3800 4000 0    50   Input ~ 0
 RPZW_IO2
+$Comp
+L Switch:SW_Push SW?
+U 1 1 608751BA
+P 7250 4900
+AR Path="/60760232/608751BA" Ref="SW?"  Part="1"
+AR Path="/60805E76/608751BA" Ref="SW1"  Part="1"
+F 0 "SW1" V 7204 5048 50  0000 L CNN
+F 1 "SW_Push" V 7295 5048 50  0000 L CNN
+F 2 "Button_Switch_THT:SW_PUSH-12mm" H 7250 5100 50  0001 C CNN
+F 3 "~" H 7250 5100 50  0001 C CNN
+	1    7250 4900
+	0    1    1    0
+$EndComp
+Wire Wire Line
+	7250 5150 7150 5150
+Connection ~ 7250 5150
+Wire Wire Line
+	7250 5150 7250 5100
+Text Label 7150 5150 2    50   ~ 0
+Button_RPZW
+$Comp
+L power:+3.3V #PWR?
+U 1 1 608751C4
+P 7250 4700
+AR Path="/608751C4" Ref="#PWR?"  Part="1"
+AR Path="/60760232/608751C4" Ref="#PWR?"  Part="1"
+AR Path="/60805E76/608751C4" Ref="#PWR0160"  Part="1"
+F 0 "#PWR0160" H 7250 4550 50  0001 C CNN
+F 1 "+3.3V" H 7265 4873 50  0000 C CNN
+F 2 "" H 7250 4700 50  0001 C CNN
+F 3 "" H 7250 4700 50  0001 C CNN
+	1    7250 4700
+	1    0    0    -1
+$EndComp
+Wire Wire Line
+	7250 5200 7250 5150
+$Comp
+L power:GND #PWR?
+U 1 1 608751CB
+P 7250 5500
+AR Path="/608751CB" Ref="#PWR?"  Part="1"
+AR Path="/607B7D6E/608751CB" Ref="#PWR?"  Part="1"
+AR Path="/60760232/608751CB" Ref="#PWR?"  Part="1"
+AR Path="/60805E76/608751CB" Ref="#PWR0161"  Part="1"
+F 0 "#PWR0161" H 7250 5250 50  0001 C CNN
+F 1 "GND" H 7255 5327 50  0000 C CNN
+F 2 "" H 7250 5500 50  0001 C CNN
+F 3 "" H 7250 5500 50  0001 C CNN
+	1    7250 5500
+	1    0    0    -1
+$EndComp
+$Comp
+L Device:R R?
+U 1 1 608751D1
+P 7250 5350
+AR Path="/6081C49D/608751D1" Ref="R?"  Part="1"
+AR Path="/607B7D6E/608751D1" Ref="R?"  Part="1"
+AR Path="/60760232/608751D1" Ref="R?"  Part="1"
+AR Path="/60805E76/608751D1" Ref="R20"  Part="1"
+F 0 "R20" V 7043 5350 50  0000 C CNN
+F 1 "1k" V 7134 5350 50  0000 C CNN
+F 2 "Resistor_SMD:R_0805_2012Metric" V 7180 5350 50  0001 C CNN
+F 3 "~" H 7250 5350 50  0001 C CNN
+	1    7250 5350
+	-1   0    0    1
+$EndComp
+Text Label 6450 4400 2    50   ~ 0
+Button_RPZW
+Wire Wire Line
+	6000 4400 6450 4400
 $EndSCHEMATC

Commit message: Archivos KiCad
Parts:
- D6: value LED -> LED_RPZW
- SW1: footprint Button_Switch_THT:SW_PUSH-12mm -> Button_Switch_THT:SW_PUSH_6mm_H4.3mm
Changed lines of the file:
@@
 AR Path="/60805E76/607E283D" Ref="D6"  Part="1"
 F 0 "D6" H 6150 5350 50  0000 C CNN
-F 1 "LED" H 6150 5250 50  0000 C CNN
+F 1 "LED_RPZW" H 6150 5250 50  0000 C CNN
 F 2 "LED_SMD:LED_0805_2012Metric" H 6150 5100 50  0001 C CNN
 F 3 "~" H 6150 5100 50  0001 C CNN
@@
 F 0 "SW1" V 7204 5048 50  0000 L CNN
 F 1 "SW_Push" V 7295 5048 50  0000 L CNN
-F 2 "Button_Switch_THT:SW_PUSH-12mm" H 7250 5100 50  0001 C CNN
+F 2 "Button_Switch_THT:SW_PUSH_6mm_H4.3mm" H 7250 5100 50  0001 C CNN
 F 3 "~" H 7250 5100 50  0001 C CNN
 	1    7250 4900

Commit message: Archivos KiCad
Parts:
- added J13: RPZW_RST, Connector_PinHeader_2.54mm:PinHeader_1x02_P2.54mm_Vertical, symbol Connector:Screw_Terminal_01x02
- added SW2: RPZW_RST_Push, Button_Switch_THT:SW_PUSH_6mm_H4.3mm, symbol Switch:SW_Push
- renumbered R10 to R11
Connections:
- new net: J13.2 (Pin_2), SW2.1
- new net: J13.1 (Pin_1), SW2.2
Other:
- moved on the sheet: R20, SW1
Changed lines of the file:
@@
 AR Path="/607B7D6E/607E2837" Ref="R?"  Part="1"
 AR Path="/60760232/607E2837" Ref="R?"  Part="1"
-AR Path="/60805E76/607E2837" Ref="R10"  Part="1"
-F 0 "R10" V 5943 4800 50  0000 C CNN
+AR Path="/60805E76/607E2837" Ref="R11"  Part="1"
+F 0 "R11" V 5943 4800 50  0000 C CNN
 F 1 "1k" V 6034 4800 50  0000 C CNN
 F 2 "Resistor_SMD:R_0805_2012Metric" V 6080 4800 50  0001 C CNN
@@
 L Switch:SW_Push SW?
 U 1 1 608751BA
-P 7250 4900
+P 7500 4900
 AR Path="/60760232/608751BA" Ref="SW?"  Part="1"
 AR Path="/60805E76/608751BA" Ref="SW1"  Part="1"
-F 0 "SW1" V 7204 5048 50  0000 L CNN
-F 1 "SW_Push" V 7295 5048 50  0000 L CNN
-F 2 "Button_Switch_THT:SW_PUSH_6mm_H4.3mm" H 7250 5100 50  0001 C CNN
-F 3 "~" H 7250 5100 50  0001 C CNN
-	1    7250 4900
+F 0 "SW1" V 7454 5048 50  0000 L CNN
+F 1 "SW_Push" V 7545 5048 50  0000 L CNN
+F 2 "Button_Switch_THT:SW_PUSH_6mm_H4.3mm" H 7500 5100 50  0001 C CNN
+F 3 "~" H 7500 5100 50  0001 C CNN
+	1    7500 4900
 	0    1    1    0
 $EndComp
 Wire Wire Line
-	7250 5150 7150 5150
-Connection ~ 7250 5150
+	7500 5150 7400 5150
+Connection ~ 7500 5150
 Wire Wire Line
-	7250 5150 7250 5100
-Text Label 7150 5150 2    50   ~ 0
+	7500 5150 7500 5100
+Text Label 7400 5150 2    50   ~ 0
 Button_RPZW
 $Comp
 L power:+3.3V #PWR?
 U 1 1 608751C4
-P 7250 4700
+P 7500 4700
 AR Path="/608751C4" Ref="#PWR?"  Part="1"
 AR Path="/60760232/608751C4" Ref="#PWR?"  Part="1"
 AR Path="/60805E76/608751C4" Ref="#PWR0160"  Part="1"
-F 0 "#PWR0160" H 7250 4550 50  0001 C CNN
-F 1 "+3.3V" H 7265 4873 50  0000 C CNN
-F 2 "" H 7250 4700 50  0001 C CNN
-F 3 "" H 7250 4700 50  0001 C CNN
-	1    7250 4700
+F 0 "#PWR0160" H 7500 4550 50  0001 C CNN
+F 1 "+3.3V" H 7515 4873 50  0000 C CNN
+F 2 "" H 7500 4700 50  0001 C CNN
+F 3 "" H 7500 4700 50  0001 C CNN
+	1    7500 4700
 	1    0    0    -1
 $EndComp
 Wire Wire Line
-	7250 5200 7250 5150
+	7500 5200 7500 5150
 $Comp
 L power:GND #PWR?
 U 1 1 608751CB
-P 7250 5500
+P 7500 5500
 AR Path="/608751CB" Ref="#PWR?"  Part="1"
 AR Path="/607B7D6E/608751CB" Ref="#PWR?"  Part="1"
 AR Path="/60760232/608751CB" Ref="#PWR?"  Part="1"
 AR Path="/60805E76/608751CB" Ref="#PWR0161"  Part="1"
-F 0 "#PWR0161" H 7250 5250 50  0001 C CNN
-F 1 "GND" H 7255 5327 50  0000 C CNN
-F 2 "" H 7250 5500 50  0001 C CNN
-F 3 "" H 7250 5500 50  0001 C CNN
-	1    7250 5500
+F 0 "#PWR0161" H 7500 5250 50  0001 C CNN
+F 1 "GND" H 7505 5327 50  0000 C CNN
+F 2 "" H 7500 5500 50  0001 C CNN
+F 3 "" H 7500 5500 50  0001 C CNN
+	1    7500 5500
 	1    0    0    -1
 $EndComp
@@
 L Device:R R?
 U 1 1 608751D1
-P 7250 5350
+P 7500 5350
 AR Path="/6081C49D/608751D1" Ref="R?"  Part="1"
 AR Path="/607B7D6E/608751D1" Ref="R?"  Part="1"
 AR Path="/60760232/608751D1" Ref="R?"  Part="1"
 AR Path="/60805E76/608751D1" Ref="R20"  Part="1"
-F 0 "R20" V 7043 5350 50  0000 C CNN
-F 1 "1k" V 7134 5350 50  0000 C CNN
-F 2 "Resistor_SMD:R_0805_2012Metric" V 7180 5350 50  0001 C CNN
-F 3 "~" H 7250 5350 50  0001 C CNN
-	1    7250 5350
+F 0 "R20" V 7293 5350 50  0000 C CNN
+F 1 "1k" V 7384 5350 50  0000 C CNN
+F 2 "Resistor_SMD:R_0805_2012Metric" V 7430 5350 50  0001 C CNN
+F 3 "~" H 7500 5350 50  0001 C CNN
+	1    7500 5350
 	-1   0    0    1
 $EndComp
@@
 Wire Wire Line
 	6000 4400 6450 4400
+$Comp
+L Connector:Screw_Terminal_01x02 J13
+U 1 1 6089EDD0
+P 8900 5300
+F 0 "J13" V 8772 5380 50  0000 L CNN
+F 1 "RPZW_RST" V 8863 5380 50  0000 L CNN
+F 2 "Connector_PinHeader_2.54mm:PinHeader_1x02_P2.54mm_Vertical" H 8900 5300 50  0001 C CNN
+F 3 "~" H 8900 5300 50  0001 C CNN
+	1    8900 5300
+	0    1    1    0
+$EndComp
+$Comp
+L Switch:SW_Push SW?
+U 1 1 6089E2F1
+P 8850 4800
+AR Path="/60760232/6089E2F1" Ref="SW?"  Part="1"
+AR Path="/60805E76/6089E2F1" Ref="SW2"  Part="1"
+F 0 "SW2" V 8804 4948 50  0000 L CNN
+F 1 "RPZW_RST_Push" V 8895 4948 50  0000 L CNN
+F 2 "Button_Switch_THT:SW_PUSH_6mm_H4.3mm" H 8850 5000 50  0001 C CNN
+F 3 "~" H 8850 5000 50  0001 C CNN
+	1    8850 4800
+	1    0    0    -1
+$EndComp
+Wire Wire Line
+	9050 4800 9050 5100
+Wire Wire Line
+	9050 5100 8900 5100
+Wire Wire Line
+	8650 4800 8650 5100
+Wire Wire Line
+	8650 5100 8800 5100
 $EndSCHEMATC

Commit message: Archivos KiCad
Connections:
- net RPWZ_JNTRST: now also J2.11 (GPIO17); no longer J2.15 (GPIO22)
- net RPWZ_JTCK: now also J2.21 (GPIO09_SPI_MISO); no longer J2.22 (GPIO25)
- net RPWZ_JTDI: now also J2.19 (GPIO10_SPI_MOSI); no longer J2.37 (GPIO26)
- net RPWZ_JTDO: now also J2.15 (GPIO22); no longer J2.18 (GPIO24)
- net RPWZ_JTMS: now also J2.23 (GPIO11_SPI_CLK); no longer J2.13 (GPIO27)
Changed lines of the file:
@@
 Text Label 3800 2700 0    50   ~ 0
 SDA_I2C
-Wire Wire Line
-	4100 4400 3800 4400
-Text Label 3900 4400 0    50   ~ 0
+Text Label 3850 3500 0    50   ~ 0
 JTDI
 Wire Wire Line
 	4100 3300 3800 3300
-Text Label 3850 3300 0    50   ~ 0
+Text Label 3850 3100 0    50   ~ 0
 JNTRST
-Wire Wire Line
-	4100 3200 3800 3200
-Text Label 3850 3200 0    50   ~ 0
+Text Label 3850 3700 0    50   ~ 0
 JTMS
 Wire Wire Line
@@
 Wire Wire Line
 	4100 2700 3800 2700
-Wire Wire Line
-	6000 2900 6300 2900
-Wire Wire Line
-	6000 3000 6300 3000
-Text Label 6100 2900 0    50   ~ 0
-TX
-Wire Wire Line
-	6000 3400 6300 3400
-Text Label 6100 3400 0    50   ~ 0
+Text Label 3850 3300 0    50   ~ 0
 JTDO
-Wire Wire Line
-	6000 3600 6300 3600
-Text Label 6100 3600 0    50   ~ 0
+Text Label 3850 3600 0    50   ~ 0
 JTCK
-Text Label 6100 3000 0    50   ~ 0
-RX
-Text HLabel 6300 3400 2    50   Input ~ 0
+Text HLabel 3800 3300 0    50   Input ~ 0
 RPWZ_JTDO
-Text HLabel 6300 3600 2    50   Input ~ 0
+Text HLabel 3800 3600 0    50   Input ~ 0
 RPWZ_JTCK
-Text HLabel 3800 4400 0    50   Input ~ 0
+Text HLabel 3800 3500 0    50   Input ~ 0
 RPWZ_JTDI
-Text HLabel 3800 3300 0    50   Input ~ 0
+Text HLabel 3800 3100 0    50   Input ~ 0
 RPWZ_JNTRST
-Text HLabel 3800 3200 0    50   Input ~ 0
+Text HLabel 3800 3700 0    50   Input ~ 0
 RPWZ_JTMS
 Text HLabel 3800 2800 0    50   Input ~ 0
@@
 Text HLabel 3800 2700 0    50   Input ~ 0
 RPWZ_SDA_I2C
-Text HLabel 6300 2900 2    50   Input ~ 0
-RPWZ_TX
-Text HLabel 6300 3000 2    50   Input ~ 0
-RPWZ_RX
 Wire Wire Line
 	4100 4200 3800 4200
@@
 Wire Wire Line
 	8650 5100 8800 5100
+Wire Wire Line
+	6000 2900 6300 2900
+Wire Wire Line
+	6000 3000 6300 3000
+Text Label 6100 2900 0    50   ~ 0
+TX
+Text HLabel 6300 2900 2    50   Input ~ 0
+RPWZ_TX
+Text Label 6100 3000 0    50   ~ 0
+RX
+Text HLabel 6300 3000 2    50   Input ~ 0
+RPWZ_RX
+Wire Wire Line
+	3800 3500 4100 3500
+Wire Wire Line
+	4100 3600 3800 3600
+Wire Wire Line
+	3800 3700 4100 3700
+Wire Wire Line
+	3800 3100 4100 3100
 $EndSCHEMATC

Commit message: Archivos KiCad
Parts:
- renumbered J13 to J11, R20 to R19
Changed lines of the file:
@@
 AR Path="/607B7D6E/608751D1" Ref="R?"  Part="1"
 AR Path="/60760232/608751D1" Ref="R?"  Part="1"
-AR Path="/60805E76/608751D1" Ref="R20"  Part="1"
-F 0 "R20" V 7293 5350 50  0000 C CNN
+AR Path="/60805E76/608751D1" Ref="R19"  Part="1"
+F 0 "R19" V 7293 5350 50  0000 C CNN
 F 1 "1k" V 7384 5350 50  0000 C CNN
 F 2 "Resistor_SMD:R_0805_2012Metric" V 7430 5350 50  0001 C CNN
@@
 	6000 4400 6450 4400
 $Comp
-L Connector:Screw_Terminal_01x02 J13
+L Connector:Screw_Terminal_01x02 J11
 U 1 1 6089EDD0
 P 8900 5300
-F 0 "J13" V 8772 5380 50  0000 L CNN
+F 0 "J11" V 8772 5380 50  0000 L CNN
 F 1 "RPZW_RST" V 8863 5380 50  0000 L CNN
 F 2 "Connector_PinHeader_2.54mm:PinHeader_1x02_P2.54mm_Vertical" H 8900 5300 50  0001 C CNN
