File: RPi_Zero_pHat_Template-master/RPi_Zero_pHat_Template.sch (KiCad schematic (older format))
At the start: 4 parts, among them U1 STM32F103C8Tx

Commit message: Archivos KiCad
Parts:
- removed L1: L, Inductor_SMD:L_0805_2012Metric, symbol Device:L
- removed R1, R2: 4.7k, Resistor_SMD:R_0805_2012Metric, symbol Device:R
- removed U1: STM32F103C8Tx, Package_QFP:LQFP-48_7x7mm_P0.5mm, symbol MCU_ST_STM32F1:STM32F103C8Tx

Commit message: Archivos KiCad
Parts:
- added J10: Test Points, Connector_PinHeader_2.54mm:PinHeader_1x07_P2.54mm_Vertical, symbol Connector:Conn_01x07_Male
- added J11: JTAG Conn, Connector_PinHeader_2.54mm:PinHeader_1x05_P2.54mm_Vertical, symbol Connector:Conn_01x05_Male
Connections:
- net DHT22: now also J10.7 (Pin_7)
- net HD38: now also J10.6 (Pin_6)
- net JNTRST: now also J11.4 (Pin_4)
- net JTCK: now also J11.2 (Pin_2)
- net JTDI: now also J11.3 (Pin_3)
- net JTDO: now also J11.1 (Pin_1)
- net JTMS: now also J11.5 (Pin_5)
- net LM35: now also J10.5 (Pin_5)
- new net +12V: J10.2 (Pin_2)
- new net +3V3: J10.4 (Pin_4)
- new net +5V: J10.3 (Pin_3)
- new net GND: J10.1 (Pin_1)
Changed lines of the file:
@@
 $EndSheet
 $Sheet
-S 2550 3250 1550 1950
+S 2550 3250 1550 2250
 U 60805E76
 F0 "RPWZ_comm" 50
@@
 F11 "RPZW_NRST" I R 4100 4100 50
 F12 "RPWZ_BOOT" I R 4100 4200 50
+F13 "RPZW_IO2" I R 4100 5250 50
+F14 "RPZW_IO1" I R 4100 5350 50
 $EndSheet
 Text Label 4650 3400 2    50   ~ 0
@@
 BOOT
 $Sheet
-S 5200 3250 1650 1950
+S 5200 3250 1650 2250
 U 60760232
 F0 "STM32" 50
@@
 F18 "STM32_JTDI" I L 5200 3600 50
 F19 "STM32_JNTRST" I L 5200 3700 50
+F20 "STM32_IO1" I L 5200 5250 50
+F21 "STM32_IO2" I L 5200 5350 50
 $EndSheet
 Wire Wire Line
@@
 Text Label 7600 4450 2    50   ~ 0
 DHT22
+Wire Wire Line
+	4100 5250 5200 5250
+Wire Wire Line
+	5200 5350 4100 5350
+Text Label 4650 5250 2    50   ~ 0
+I_O_1
+Text Label 4650 5350 2    50   ~ 0
+I_O_2
+$Comp
+L power:+12V #PWR0155
+U 1 1 60862CC1
+P 4400 6550
+F 0 "#PWR0155" H 4400 6400 50  0001 C CNN
+F 1 "+12V" V 4415 6678 50  0000 L CNN
+F 2 "" H 4400 6550 50  0001 C CNN
+F 3 "" H 4400 6550 50  0001 C CNN
+	1    4400 6550
+	0    1    1    0
+$EndComp
+Wire Wire Line
+	4400 6550 4150 6550
+$Comp
+L power:+5V #PWR0156
+U 1 1 60863A5B
+P 4400 6650
+F 0 "#PWR0156" H 4400 6500 50  0001 C CNN
+F 1 "+5V" V 4415 6778 50  0000 L CNN
+F 2 "" H 4400 6650 50  0001 C CNN
+F 3 "" H 4400 6650 50  0001 C CNN
+	1    4400 6650
+	0    1    1    0
+$EndComp
+Wire Wire Line
+	4400 6650 4150 6650
+Wire Wire Line
+	4400 6750 4150 6750
+Text Label 4500 6850 2    50   ~ 0
+LM35
+$Comp
+L power:+3.3V #r0101
+U 1 1 60864648
+P 4400 6750
+F 0 "#r0101" H 4400 6600 50  0001 C CNN
+F 1 "+3.3V" V 4415 6878 50  0000 L CNN
+F 2 "" H 4400 6750 50  0001 C CNN
+F 3 "" H 4400 6750 50  0001 C CNN
+	1    4400 6750
+	0    1    1    0
+$EndComp
+Wire Wire Line
+	4150 6850 4500 6850
+Wire Wire Line
+	4150 6950 4500 6950
+Wire Wire Line
+	4150 7050 4500 7050
+Text Label 4500 6950 2    50   ~ 0
+HD38
+Text Label 4500 7050 2    50   ~ 0
+DHT22
+$Comp
+L Connector:Conn_01x07_Male J10
+U 1 1 60867F6C
+P 3950 6750
+F 0 "J10" H 4058 7231 50  0000 C CNN
+F 1 "Test Points" H 4058 7140 50  0000 C CNN
+F 2 "Connector_PinHeader_2.54mm:PinHeader_1x07_P2.54mm_Vertical" H 3950 6750 50  0001 C CNN
+F 3 "~" H 3950 6750 50  0001 C CNN
+	1    3950 6750
+	1    0    0    -1
+$EndComp
+$Comp
+L power:GND #PWR0157
+U 1 1 6086B115
+P 4400 6450
+F 0 "#PWR0157" H 4400 6200 50  0001 C CNN
+F 1 "GND" V 4405 6322 50  0000 R CNN
+F 2 "" H 4400 6450 50  0001 C CNN
+F 3 "" H 4400 6450 50  0001 C CNN
+	1    4400 6450
+	0    -1   -1   0
+$EndComp
+Wire Wire Line
+	4400 6450 4150 6450
+$Comp
+L Connector:Conn_01x05_Male J11
+U 1 1 60870978
+P 5650 6600
+F 0 "J11" H 5758 6981 50  0000 C CNN
+F 1 "JTAG Conn" H 5758 6890 50  0000 C CNN
+F 2 "Connector_PinHeader_2.54mm:PinHeader_1x05_P2.54mm_Vertical" H 5650 6600 50  0001 C CNN
+F 3 "~" H 5650 6600 50  0001 C CNN
+	1    5650 6600
+	1    0    0    -1
+$EndComp
+Wire Wire Line
+	5850 6400 6300 6400
+Text Label 6300 6400 2    50   ~ 0
+JTDO
+Wire Wire Line
+	5850 6500 6300 6500
+Wire Wire Line
+	5850 6600 6300 6600
+Wire Wire Line
+	5850 6700 6300 6700
+Wire Wire Line
+	5850 6800 6300 6800
+Text Label 6300 6500 2    50   ~ 0
+JTCK
+Text Label 6300 6600 2    50   ~ 0
+JTDI
+Text Label 6300 6700 2    50   ~ 0
+JNTRST
+Text Label 6300 6800 2    50   ~ 0
+JTMS
 $EndSCHEMATC

Commit message: Archivos KiCad
Parts:
- removed J11: JTAG Conn, Connector_PinHeader_2.54mm:PinHeader_1x05_P2.54mm_Vertical, symbol Connector:Conn_01x05_Male
Changed lines of the file:
@@
 Wire Wire Line
 	4400 6450 4150 6450
-$Comp
-L Connector:Conn_01x05_Male J11
-U 1 1 60870978
-P 5650 6600
-F 0 "J11" H 5758 6981 50  0000 C CNN
-F 1 "JTAG Conn" H 5758 6890 50  0000 C CNN
-F 2 "Connector_PinHeader_2.54mm:PinHeader_1x05_P2.54mm_Vertical" H 5650 6600 50  0001 C CNN
-F 3 "~" H 5650 6600 50  0001 C CNN
-	1    5650 6600
-	1    0    0    -1
-$EndComp
-Wire Wire Line
-	5850 6400 6300 6400
-Text Label 6300 6400 2    50   ~ 0
-JTDO
-Wire Wire Line
-	5850 6500 6300 6500
-Wire Wire Line
-	5850 6600 6300 6600
-Wire Wire Line
-	5850 6700 6300 6700
-Wire Wire Line
-	5850 6800 6300 6800
-Text Label 6300 6500 2    50   ~ 0
-JTCK
-Text Label 6300 6600 2    50   ~ 0
-JTDI
-Text Label 6300 6700 2    50   ~ 0
-JNTRST
-Text Label 6300 6800 2    50   ~ 0
-JTMS
 $EndSCHEMATC

Commit message: Archivos KiCad
Parts:
- J10: footprint Connector_PinHeader_2.54mm:PinHeader_1x07_P2.54mm_Vertical -> Connector_PinHeader_2.54mm:PinHeader_1x06_P2.54mm_Vertical; symbol Connector:Conn_01x07_Male -> Connector:Conn_01x06_Male
Connections:
- net LM35 is gone; now on net HD38: J10.5 (Pin_5)
- net DHT22: now also J10.6 (Pin_6); no longer J10.7 (Pin_7)
- net HD38: no longer J10.6 (Pin_6)
Changed lines of the file:
@@
 F0 "In_Out" 50
 F1 "In_Out.sch" 50
-F2 "Out_LM35" I L 7850 4250 50
-F3 "Out_DHT22" I L 7850 4450 50
-F4 "Out_HD38" I L 7850 4350 50
-F5 "In_Resistencia_Si" I L 7850 3600 50
-F6 "In_Ventilador" I L 7850 3700 50
-F7 "In_Bomba_Agua" I L 7850 3800 50
-F8 "In_LEDs" I L 7850 3900 50
+F2 "Out_DHT22" I L 7850 4450 50
+F3 "Out_HD38" I L 7850 4350 50
+F4 "In_Resistencia_Si" I L 7850 3600 50
+F5 "In_Ventilador" I L 7850 3700 50
+F6 "In_Bomba_Agua" I L 7850 3800 50
+F7 "In_LEDs" I L 7850 3900 50
 $EndSheet
 Text Label 4650 4100 2    50   ~ 0
@@
 F9 "STM32_Bomba_Agua" I R 6850 3800 50
 F10 "STM32_LEDs" I R 6850 3900 50
-F11 "STM32_LM35" I R 6850 4250 50
-F12 "STM32_HD38" I R 6850 4350 50
-F13 "STM32_DHT22" I R 6850 4450 50
-F14 "STM32_TX" I L 5200 5000 50
-F15 "STM32_RX" I L 5200 4900 50
-F16 "STM32_JTMS" I L 5200 3800 50
-F17 "STM32_JTCK" I L 5200 3500 50
-F18 "STM32_JTDI" I L 5200 3600 50
-F19 "STM32_JNTRST" I L 5200 3700 50
-F20 "STM32_IO1" I L 5200 5250 50
-F21 "STM32_IO2" I L 5200 5350 50
+F11 "STM32_HD38" I R 6850 4350 50
+F12 "STM32_DHT22" I R 6850 4450 50
+F13 "STM32_TX" I L 5200 5000 50
+F14 "STM32_RX" I L 5200 4900 50
+F15 "STM32_JTMS" I L 5200 3800 50
+F16 "STM32_JTCK" I L 5200 3500 50
+F17 "STM32_JTDI" I L 5200 3600 50
+F18 "STM32_JNTRST" I L 5200 3700 50
+F19 "STM32_IO1" I L 5200 5250 50
+F20 "STM32_IO2" I L 5200 5350 50
 $EndSheet
 Wire Wire Line
@@
 	6850 3900 7850 3900
 Wire Wire Line
-	7850 4250 6850 4250
-Wire Wire Line
 	6850 4350 7850 4350
 Wire Wire Line
@@
 Text Label 7600 3900 2    50   ~ 0
 LEDs
-Text Label 7600 4250 2    50   ~ 0
-LM35
 Text Label 7600 4350 2    50   ~ 0
 HD38
@@
 Wire Wire Line
 	4400 6750 4150 6750
-Text Label 4500 6850 2    50   ~ 0
-LM35
 $Comp
 L power:+3.3V #r0101
@@
 	0    1    1    0
 $EndComp
-Wire Wire Line
-	4150 6850 4500 6850
-Wire Wire Line
-	4150 6950 4500 6950
-Wire Wire Line
-	4150 7050 4500 7050
+Text Label 4500 6850 2    50   ~ 0
+HD38
 Text Label 4500 6950 2    50   ~ 0
-HD38
-Text Label 4500 7050 2    50   ~ 0
 DHT22
 $Comp
-L Connector:Conn_01x07_Male J10
+L Connector:Conn_01x06_Male J10
 U 1 1 60867F6C
-P 3950 6750
-F 0 "J10" H 4058 7231 50  0000 C CNN
-F 1 "Test Points" H 4058 7140 50  0000 C CNN
-F 2 "Connector_PinHeader_2.54mm:PinHeader_1x07_P2.54mm_Vertical" H 3950 6750 50  0001 C CNN
-F 3 "~" H 3950 6750 50  0001 C CNN
-	1    3950 6750
+P 3950 6650
+F 0 "J10" H 4058 7131 50  0000 C CNN
+F 1 "Test Points" H 4058 7040 50  0000 C CNN
+F 2 "Connector_PinHeader_2.54mm:PinHeader_1x06_P2.54mm_Vertical" H 3950 6650 50  0001 C CNN
+F 3 "~" H 3950 6650 50  0001 C CNN
+	1    3950 6650
 	1    0    0    -1
 $EndComp
@@
 Wire Wire Line
 	4400 6450 4150 6450
+Wire Wire Line
+	4150 6850 4500 6850
+Wire Wire Line
+	4500 6950 4150 6950
 $EndSCHEMATC
