File: RPi_Zero_pHat_Template-master/STM32.sch (KiCad schematic (older format))
At the start: 13 parts, among them U1 STM32F103C8Tx

Commit message: Archivos KiCad
Parts:
- added D5: LED, LED_SMD:LED_0805_2012Metric, symbol Device:LED
- added R11: 1k, Resistor_SMD:R_0805_2012Metric, symbol Device:R
Connections:
- net GND: now also D5.1 (K)
- net STM32_Bomba_Agua: now also U1.42 (PB6); no longer U1.13 (PA3)
- net STM32_LEDs: now also U1.41 (PB5); no longer U1.14 (PA4)
- net STM32_Resistencia_Si: now also U1.45 (PB8); no longer U1.11 (PA1)
- net STM32_Ventilador: now also U1.43 (PB7); no longer U1.12 (PA2)
- net at U1.46 (PB9): now also R11.1
- new net: D5.2 (A), R11.2
Changed lines of the file:
@@
 BOOT
 Wire Wire Line
-	5150 3550 4150 3550
-Wire Wire Line
-	5150 3650 4150 3650
-Wire Wire Line
-	5150 3750 4150 3750
-Wire Wire Line
-	5150 3850 4150 3850
-Wire Wire Line
 	5150 3950 4150 3950
 Wire Wire Line
@@
 Wire Wire Line
 	5150 4150 4150 4150
-Text Label 4250 3550 0    50   ~ 0
+Text Label 2150 4250 0    50   ~ 0
 O_Resistencia_Si
-Text Label 4250 3650 0    50   ~ 0
+Text Label 2150 4150 0    50   ~ 0
 O_Ventilador
-Text Label 4250 3750 0    50   ~ 0
+Text Label 2150 4050 0    50   ~ 0
 O_Bomba_Agua
-Text Label 4250 3850 0    50   ~ 0
+Text Label 2150 3950 0    50   ~ 0
 O_LEDs
 Text Label 4250 3950 0    50   ~ 0
@@
 Text HLabel 8350 2000 2    50   Input ~ 0
 STM32_SDA_I2C
-Text HLabel 5150 3550 2    50   Input ~ 0
+Text HLabel 2050 4250 0    50   Input ~ 0
 STM32_Resistencia_Si
-Text HLabel 5150 3650 2    50   Input ~ 0
+Text HLabel 2050 4150 0    50   Input ~ 0
 STM32_Ventilador
-Text HLabel 5150 3750 2    50   Input ~ 0
+Text HLabel 2050 4050 0    50   Input ~ 0
 STM32_Bomba_Agua
-Text HLabel 5150 3850 2    50   Input ~ 0
+Text HLabel 2050 3950 0    50   Input ~ 0
 STM32_LEDs
 Text HLabel 5150 3950 2    50   Input ~ 0
@@
 Text Label 8000 4450 0    50   ~ 0
 VDDA
+Wire Wire Line
+	2850 3950 2050 3950
+Wire Wire Line
+	2050 4050 2850 4050
+Wire Wire Line
+	2050 4150 2850 4150
+Wire Wire Line
+	2050 4250 2850 4250
+$Comp
+L Device:R R?
+U 1 1 607A4463
+P 2000 4600
+AR Path="/6081C49D/607A4463" Ref="R?"  Part="1"
+AR Path="/607B7D6E/607A4463" Ref="R?"  Part="1"
+AR Path="/60760232/607A4463" Ref="R11"  Part="1"
+F 0 "R11" V 1793 4600 50  0000 C CNN
+F 1 "1k" V 1884 4600 50  0000 C CNN
+F 2 "Resistor_SMD:R_0805_2012Metric" V 1930 4600 50  0001 C CNN
+F 3 "~" H 2000 4600 50  0001 C CNN
+	1    2000 4600
+	1    0    0    -1
+$EndComp
+$Comp
+L Device:LED D?
+U 1 1 607A446A
+P 2000 4900
+AR Path="/607B7D6E/607A446A" Ref="D?"  Part="1"
+AR Path="/60760232/607A446A" Ref="D5"  Part="1"
+F 0 "D5" H 2000 5150 50  0000 C CNN
+F 1 "LED" H 2000 5050 50  0000 C CNN
+F 2 "LED_SMD:LED_0805_2012Metric" H 2000 4900 50  0001 C CNN
+F 3 "~" H 2000 4900 50  0001 C CNN
+	1    2000 4900
+	0    -1   -1   0
+$EndComp
+Wire Wire Line
+	2000 5100 2000 5050
+$Comp
+L power:GND #PWR?
+U 1 1 607A4473
+P 2000 5100
+AR Path="/607A4473" Ref="#PWR?"  Part="1"
+AR Path="/607B7D6E/607A4473" Ref="#PWR?"  Part="1"
+AR Path="/60760232/607A4473" Ref="#PWR0148"  Part="1"
+F 0 "#PWR0148" H 2000 4850 50  0001 C CNN
+F 1 "GND" H 2005 4927 50  0000 C CNN
+F 2 "" H 2000 5100 50  0001 C CNN
+F 3 "" H 2000 5100 50  0001 C CNN
+	1    2000 5100
+	1    0    0    -1
+$EndComp
+Wire Wire Line
+	2000 4450 2000 4350
+Wire Wire Line
+	2000 4350 2850 4350
 $EndSCHEMATC

Commit message: Archivos KiCad
Parts:
- C1, C11, C4, C5, C6, C7: footprint Capacitor_SMD:C_0805_2012Metric -> Capacitor_SMD:C_0603_1608Metric
- C8: footprint Capacitor_SMD:C_0805_2012Metric -> Capacitor_SMD:C_0402_1005Metric
- L1, L2: value L -> 33nH; footprint Inductor_SMD:L_0805_2012Metric -> Inductor_SMD:L_0402_1005Metric
Changed lines of the file:
@@
 AR Path="/60760232/60762529" Ref="L1"  Part="1"
 F 0 "L1" V 4040 5200 50  0000 C CNN
-F 1 "L" V 3949 5200 50  0000 C CNN
-F 2 "Inductor_SMD:L_0805_2012Metric" H 3850 5200 50  0001 C CNN
+F 1 "33nH" V 3949 5200 50  0000 C CNN
+F 2 "Inductor_SMD:L_0402_1005Metric" H 3850 5200 50  0001 C CNN
 F 3 "~" H 3850 5200 50  0001 C CNN
 	1    3850 5200
@@
 F 0 "C1" H 6865 3196 50  0000 L CNN
 F 1 "100nF" H 6865 3105 50  0000 L CNN
-F 2 "Capacitor_SMD:C_0805_2012Metric" H 6788 3000 50  0001 C CNN
+F 2 "Capacitor_SMD:C_0603_1608Metric" H 6788 3000 50  0001 C CNN
 F 3 "~" H 6750 3150 50  0001 C CNN
 	1    6750 3150
@@
 F 0 "C4" H 7365 3196 50  0000 L CNN
 F 1 "100nF" H 7365 3105 50  0000 L CNN
-F 2 "Capacitor_SMD:C_0805_2012Metric" H 7288 3000 50  0001 C CNN
+F 2 "Capacitor_SMD:C_0603_1608Metric" H 7288 3000 50  0001 C CNN
 F 3 "~" H 7250 3150 50  0001 C CNN
 	1    7250 3150
@@
 F 0 "C5" H 7865 3196 50  0000 L CNN
 F 1 "100nF" H 7865 3105 50  0000 L CNN
-F 2 "Capacitor_SMD:C_0805_2012Metric" H 7788 3000 50  0001 C CNN
+F 2 "Capacitor_SMD:C_0603_1608Metric" H 7788 3000 50  0001 C CNN
 F 3 "~" H 7750 3150 50  0001 C CNN
 	1    7750 3150
@@
 F 0 "C7" H 8365 3196 50  0000 L CNN
 F 1 "100nF" H 8365 3105 50  0000 L CNN
-F 2 "Capacitor_SMD:C_0805_2012Metric" H 8288 3000 50  0001 C CNN
+F 2 "Capacitor_SMD:C_0603_1608Metric" H 8288 3000 50  0001 C CNN
 F 3 "~" H 8250 3150 50  0001 C CNN
 	1    8250 3150
@@
 F 0 "C11" H 8865 3196 50  0000 L CNN
 F 1 "100nF" H 8865 3105 50  0000 L CNN
-F 2 "Capacitor_SMD:C_0805_2012Metric" H 8788 3000 50  0001 C CNN
+F 2 "Capacitor_SMD:C_0603_1608Metric" H 8788 3000 50  0001 C CNN
 F 3 "~" H 8750 3150 50  0001 C CNN
 	1    8750 3150
@@
 F 0 "C6" H 7915 4796 50  0000 L CNN
 F 1 "10nF" H 7915 4705 50  0000 L CNN
-F 2 "Capacitor_SMD:C_0805_2012Metric" H 7838 4600 50  0001 C CNN
+F 2 "Capacitor_SMD:C_0603_1608Metric" H 7838 4600 50  0001 C CNN
 F 3 "~" H 7800 4750 50  0001 C CNN
 	1    7800 4750
@@
 F 0 "C8" H 8365 4796 50  0000 L CNN
 F 1 "1uF" H 8365 4705 50  0000 L CNN
-F 2 "Capacitor_SMD:C_0805_2012Metric" H 8288 4600 50  0001 C CNN
+F 2 "Capacitor_SMD:C_0402_1005Metric" H 8288 4600 50  0001 C CNN
 F 3 "~" H 8250 4750 50  0001 C CNN
 	1    8250 4750
@@
 AR Path="/60760232/6076D270" Ref="L2"  Part="1"
 F 0 "L2" V 8040 4450 50  0000 C CNN
-F 1 "L" V 7949 4450 50  0000 C CNN
-F 2 "Inductor_SMD:L_0805_2012Metric" H 7850 4450 50  0001 C CNN
+F 1 "33nH" V 7949 4450 50  0000 C CNN
+F 2 "Inductor_SMD:L_0402_1005Metric" H 7850 4450 50  0001 C CNN
 F 3 "~" H 7850 4450 50  0001 C CNN
 	1    7850 4450

Commit message: Archivos KiCad
Connections:
- net STM32_IO2: now reaches U1.18 (PB0)
- net STM32_IO1: now reaches U1.19 (PB1)
Changed lines of the file:
@@
 Wire Wire Line
 	2000 4350 2850 4350
+Wire Wire Line
+	2850 3450 2550 3450
+Wire Wire Line
+	2850 3550 2550 3550
+Text HLabel 2550 3550 0    50   Input ~ 0
+STM32_IO1
+Text HLabel 2550 3450 0    50   Input ~ 0
+STM32_IO2
 $EndSCHEMATC

Commit message: Archivos KiCad
Parts:
- added R19: 1k, Resistor_SMD:R_0805_2012Metric, symbol Device:R
- added SW3: SW_Push, Button_Switch_THT:SW_PUSH-12mm, symbol Switch:SW_Push
- C1, C11, C4, C5, C7: footprint Capacitor_SMD:C_0603_1608Metric -> Capacitor_SMD:C_0201_0603Metric
- C6: footprint Capacitor_SMD:C_0603_1608Metric -> Capacitor_SMD:C_0805_2012Metric
- C8: footprint Capacitor_SMD:C_0402_1005Metric -> Capacitor_SMD:C_0805_2012Metric
Connections:
- net +3V3: now also SW3.1
- net GND: now also R19.1
- net Button_STM32: now reaches U1.25 (PB12)
- net Button_STM32: now also R19.2, SW3.2
Changed lines of the file:
@@
 F 0 "C1" H 6865 3196 50  0000 L CNN
 F 1 "100nF" H 6865 3105 50  0000 L CNN
-F 2 "Capacitor_SMD:C_0603_1608Metric" H 6788 3000 50  0001 C CNN
+F 2 "Capacitor_SMD:C_0201_0603Metric" H 6788 3000 50  0001 C CNN
 F 3 "~" H 6750 3150 50  0001 C CNN
 	1    6750 3150
@@
 F 0 "C4" H 7365 3196 50  0000 L CNN
 F 1 "100nF" H 7365 3105 50  0000 L CNN
-F 2 "Capacitor_SMD:C_0603_1608Metric" H 7288 3000 50  0001 C CNN
+F 2 "Capacitor_SMD:C_0201_0603Metric" H 7288 3000 50  0001 C CNN
 F 3 "~" H 7250 3150 50  0001 C CNN
 	1    7250 3150
@@
 F 0 "C5" H 7865 3196 50  0000 L CNN
 F 1 "100nF" H 7865 3105 50  0000 L CNN
-F 2 "Capacitor_SMD:C_0603_1608Metric" H 7788 3000 50  0001 C CNN
+F 2 "Capacitor_SMD:C_0201_0603Metric" H 7788 3000 50  0001 C CNN
 F 3 "~" H 7750 3150 50  0001 C CNN
 	1    7750 3150
@@
 F 0 "C7" H 8365 3196 50  0000 L CNN
 F 1 "100nF" H 8365 3105 50  0000 L CNN
-F 2 "Capacitor_SMD:C_0603_1608Metric" H 8288 3000 50  0001 C CNN
+F 2 "Capacitor_SMD:C_0201_0603Metric" H 8288 3000 50  0001 C CNN
 F 3 "~" H 8250 3150 50  0001 C CNN
 	1    8250 3150
@@
 F 0 "C11" H 8865 3196 50  0000 L CNN
 F 1 "100nF" H 8865 3105 50  0000 L CNN
-F 2 "Capacitor_SMD:C_0603_1608Metric" H 8788 3000 50  0001 C CNN
+F 2 "Capacitor_SMD:C_0201_0603Metric" H 8788 3000 50  0001 C CNN
 F 3 "~" H 8750 3150 50  0001 C CNN
 	1    8750 3150
@@
 F 0 "C6" H 7915 4796 50  0000 L CNN
 F 1 "10nF" H 7915 4705 50  0000 L CNN
-F 2 "Capacitor_SMD:C_0603_1608Metric" H 7838 4600 50  0001 C CNN
+F 2 "Capacitor_SMD:C_0805_2012Metric" H 7838 4600 50  0001 C CNN
 F 3 "~" H 7800 4750 50  0001 C CNN
 	1    7800 4750
@@
 F 0 "C8" H 8365 4796 50  0000 L CNN
 F 1 "1uF" H 8365 4705 50  0000 L CNN
-F 2 "Capacitor_SMD:C_0402_1005Metric" H 8288 4600 50  0001 C CNN
+F 2 "Capacitor_SMD:C_0805_2012Metric" H 8288 4600 50  0001 C CNN
 F 3 "~" H 8250 4750 50  0001 C CNN
 	1    8250 4750
@@
 Text HLabel 2550 3450 0    50   Input ~ 0
 STM32_IO2
+$Comp
+L Switch:SW_Push SW3
+U 1 1 60832580
+P 2050 6250
+F 0 "SW3" V 2004 6398 50  0000 L CNN
+F 1 "SW_Push" V 2095 6398 50  0000 L CNN
+F 2 "Button_Switch_THT:SW_PUSH-12mm" H 2050 6450 50  0001 C CNN
+F 3 "~" H 2050 6450 50  0001 C CNN
+	1    2050 6250
+	0    1    1    0
+$EndComp
+Text Label 2300 4650 0    50   ~ 0
+Button_STM32
+Wire Wire Line
+	2050 6500 1950 6500
+Connection ~ 2050 6500
+Wire Wire Line
+	2050 6500 2050 6450
+Text Label 1950 6500 2    50   ~ 0
+Button_STM32
+$Comp
+L power:+3.3V #PWR?
+U 1 1 6085D9ED
+P 2050 6050
+AR Path="/6085D9ED" Ref="#PWR?"  Part="1"
+AR Path="/60760232/6085D9ED" Ref="#PWR0158"  Part="1"
+F 0 "#PWR0158" H 2050 5900 50  0001 C CNN
+F 1 "+3.3V" H 2065 6223 50  0000 C CNN
+F 2 "" H 2050 6050 50  0001 C CNN
+F 3 "" H 2050 6050 50  0001 C CNN
+	1    2050 6050
+	1    0    0    -1
+$EndComp
+Wire Wire Line
+	2050 6550 2050 6500
+$Comp
+L power:GND #PWR?
+U 1 1 608586C0
+P 2050 6850
+AR Path="/608586C0" Ref="#PWR?"  Part="1"
+AR Path="/607B7D6E/608586C0" Ref="#PWR?"  Part="1"
+AR Path="/60760232/608586C0" Ref="#PWR0159"  Part="1"
+F 0 "#PWR0159" H 2050 6600 50  0001 C CNN
+F 1 "GND" H 2055 6677 50  0000 C CNN
+F 2 "" H 2050 6850 50  0001 C CNN
+F 3 "" H 2050 6850 50  0001 C CNN
+	1    2050 6850
+	1    0    0    -1
+$EndComp
+$Comp
+L Device:R R?
+U 1 1 6085276C
+P 2050 6700
+AR Path="/6081C49D/6085276C" Ref="R?"  Part="1"
+AR Path="/607B7D6E/6085276C" Ref="R?"  Part="1"
+AR Path="/60760232/6085276C" Ref="R19"  Part="1"
+F 0 "R19" V 1843 6700 50  0000 C CNN
+F 1 "1k" V 1934 6700 50  0000 C CNN
+F 2 "Resistor_SMD:R_0805_2012Metric" V 1980 6700 50  0001 C CNN
+F 3 "~" H 2050 6700 50  0001 C CNN
+	1    2050 6700
+	-1   0    0    1
+$EndComp
+Wire Wire Line
+	2300 4650 2850 4650
 $EndSCHEMATC

Commit message: Archivos KiCad
Parts:
- added J12: Conn_USART, TerminalBlock_Phoenix:TerminalBlock_Phoenix_MKDS-1,5-2-5.08_1x02_P5.08mm_Horizontal, symbol Connector:Screw_Terminal_01x02
- C1, C11, C4, C5, C7: footprint Capacitor_SMD:C_0201_0603Metric -> Capacitor_SMD:C_0805_2012Metric
Connections:
- net TX2: now reaches U1.12 (PA2)
- net TX2: now also J12.1 (Pin_1)
- net RX2: now reaches U1.13 (PA3)
- net RX2: now also J12.2 (Pin_2)
Changed lines of the file:
@@
 	4150 4350 4450 4350
 Text Label 4450 4350 2    50   ~ 0
-TX
+TX1
 Wire Wire Line
 	4150 4450 4450 4450
 Text Label 4450 4450 2    50   ~ 0
-RX
+RX1
 Wire Wire Line
 	4150 4750 4450 4750
@@
 F 0 "C1" H 6865 3196 50  0000 L CNN
 F 1 "100nF" H 6865 3105 50  0000 L CNN
-F 2 "Capacitor_SMD:C_0201_0603Metric" H 6788 3000 50  0001 C CNN
+F 2 "Capacitor_SMD:C_0805_2012Metric" H 6788 3000 50  0001 C CNN
 F 3 "~" H 6750 3150 50  0001 C CNN
 	1    6750 3150
@@
 F 0 "C4" H 7365 3196 50  0000 L CNN
 F 1 "100nF" H 7365 3105 50  0000 L CNN
-F 2 "Capacitor_SMD:C_0201_0603Metric" H 7288 3000 50  0001 C CNN
+F 2 "Capacitor_SMD:C_0805_2012Metric" H 7288 3000 50  0001 C CNN
 F 3 "~" H 7250 3150 50  0001 C CNN
 	1    7250 3150
@@
 F 0 "C5" H 7865 3196 50  0000 L CNN
 F 1 "100nF" H 7865 3105 50  0000 L CNN
-F 2 "Capacitor_SMD:C_0201_0603Metric" H 7788 3000 50  0001 C CNN
+F 2 "Capacitor_SMD:C_0805_2012Metric" H 7788 3000 50  0001 C CNN
 F 3 "~" H 7750 3150 50  0001 C CNN
 	1    7750 3150
@@
 F 0 "C7" H 8365 3196 50  0000 L CNN
 F 1 "100nF" H 8365 3105 50  0000 L CNN
-F 2 "Capacitor_SMD:C_0201_0603Metric" H 8288 3000 50  0001 C CNN
+F 2 "Capacitor_SMD:C_0805_2012Metric" H 8288 3000 50  0001 C CNN
 F 3 "~" H 8250 3150 50  0001 C CNN
 	1    8250 3150
@@
 F 0 "C11" H 8865 3196 50  0000 L CNN
 F 1 "100nF" H 8865 3105 50  0000 L CNN
-F 2 "Capacitor_SMD:C_0201_0603Metric" H 8788 3000 50  0001 C CNN
+F 2 "Capacitor_SMD:C_0805_2012Metric" H 8788 3000 50  0001 C CNN
 F 3 "~" H 8750 3150 50  0001 C CNN
 	1    8750 3150
@@
 Wire Wire Line
 	2300 4650 2850 4650
+$Comp
+L Connector:Screw_Terminal_01x02 J?
+U 1 1 6082711C
+P 4750 3450
+AR Path="/6081C49D/6082711C" Ref="J?"  Part="1"
+AR Path="/60760232/6082711C" Ref="J12"  Part="1"
+F 0 "J12" V 4714 3262 50  0000 R CNN
+F 1 "Conn_USART" V 4623 3262 50  0000 R CNN
+F 2 "TerminalBlock_Phoenix:TerminalBlock_Phoenix_MKDS-1,5-2-5.08_1x02_P5.08mm_Horizontal" H 4750 3450 50  0001 C CNN
+F 3 "~" H 4750 3450 50  0001 C CNN
+	1    4750 3450
+	0    -1   -1   0
+$EndComp
+Wire Wire Line
+	4150 3650 4750 3650
+Text Label 4550 3650 2    50   ~ 0
+TX2
+Wire Wire Line
+	4150 3750 4850 3750
+Wire Wire Line
+	4850 3750 4850 3650
+Text Label 4550 3750 2    50   ~ 0
+RX2
 $EndSCHEMATC

Commit message: Archivos KiCad
Parts:
- D5: value LED -> LED_STM
- J12: footprint TerminalBlock_Phoenix:TerminalBlock_Phoenix_MKDS-1,5-2-5.08_1x02_P5.08mm_Horizontal -> Connector_PinHeader_2.54mm:PinHeader_1x02_P2.54mm_Vertical
- SW3: footprint Button_Switch_THT:SW_PUSH-12mm -> Button_Switch_THT:SW_PUSH_6mm_H4.3mm

Commit message: Archivos KiCad
Parts:
- removed J12: Conn_USART, Connector_PinHeader_2.54mm:PinHeader_1x02_P2.54mm_Vertical, symbol Connector:Screw_Terminal_01x02
- removed R19: 1k, Resistor_SMD:R_0805_2012Metric, symbol Device:R
- removed SW3: SW_Push, Button_Switch_THT:SW_PUSH_6mm_H4.3mm, symbol Switch:SW_Push
- added J12: USART_Conn, Connector_PinHeader_2.54mm:PinHeader_1x03_P2.54mm_Vertical, symbol Connector:Screw_Terminal_01x03
- renumbered R11 to R10
Connections:
- net GND: now also J12.1 (Pin_1)
- net RX2: now also U1.22 (PB11), J12.2 (Pin_2); no longer U1.13 (PA3)
- net STM32_Bomba_Agua: now also U1.11 (PA1); no longer U1.42 (PB6)
- net STM32_DHT22: now also U1.15 (PA5); no longer U1.17 (PA7)
- net STM32_LEDs: now also U1.13 (PA3); no longer U1.41 (PB5)
- net STM32_LM35: now also U1.17 (PA7); no longer U1.15 (PA5)
- net STM32_Resistencia_Si: now also U1.10 (PA0); no longer U1.45 (PB8)
- net STM32_SCL_I2C: now also U1.42 (PB6); no longer U1.21 (PB10)
- net STM32_SDA_I2C: now also U1.43 (PB7); no longer U1.22 (PB11)
- net STM32_Ventilador: now also U1.12 (PA2); no longer U1.43 (PB7)
- net TX2: now also U1.21 (PB10), J12.3 (Pin_3); no longer U1.12 (PA2)
- net VSSA: now reaches L1.1, U1.8 (VSSA)
- net Button_STM32: no longer names the net of U1.25 (PB12)
Other:
- moved on the sheet: C1, C11, C12, C4, C5, C7, L1

Commit message: Archivos KiCad
Parts:
- L1, L2: footprint Inductor_SMD:L_0402_1005Metric -> Inductor_SMD:L_0603_1608Metric
Connections:
- net STM32_LM35: no longer names the net of U1.17 (PA7)
Changed lines of the file:
@@
 F 0 "L1" V 4290 5200 50  0000 C CNN
 F 1 "33nH" V 4199 5200 50  0000 C CNN
-F 2 "Inductor_SMD:L_0402_1005Metric" H 4100 5200 50  0001 C CNN
+F 2 "Inductor_SMD:L_0603_1608Metric" H 4100 5200 50  0001 C CNN
 F 3 "~" H 4100 5200 50  0001 C CNN
 	1    4100 5200
@@
 Wire Wire Line
 	5150 4050 4150 4050
-Wire Wire Line
-	5150 4150 4150 4150
 Text Label 4250 3450 0    50   ~ 0
 O_Resistencia_Si
@@
 Text Label 4250 3750 0    50   ~ 0
 O_LEDs
-Text Label 4250 4150 0    50   ~ 0
-I_LM35
 Text Label 4250 4050 0    50   ~ 0
 I_HD38
@@
 Text HLabel 5150 3750 2    50   Input ~ 0
 STM32_LEDs
-Text HLabel 5150 4150 2    50   Input ~ 0
-STM32_LM35
 Text HLabel 5150 4050 2    50   Input ~ 0
 STM32_HD38
@@
 F 0 "L2" V 8040 4450 50  0000 C CNN
 F 1 "33nH" V 7949 4450 50  0000 C CNN
-F 2 "Inductor_SMD:L_0402_1005Metric" H 7850 4450 50  0001 C CNN
+F 2 "Inductor_SMD:L_0603_1608Metric" H 7850 4450 50  0001 C CNN
 F 3 "~" H 7850 4450 50  0001 C CNN
 	1    7850 4450
